File: Hardware/Output.sch (KiCad schematic (older format))
At the start: 15 parts

Commit message: output amplifier stage finished+THS3091 added to library
Parts:
- removed U?: TLV3541, symbol OS-LD:TVL3541
- added C?: 100nF, symbol Device:C
- added R?: 750R, symbol Device:R
- added R? (x2): 25R, symbol Device:R
- added U? (x2): THS3091, symbol OS-LD:THS3091
Connections:
- net GND: now also C?.1, U?.4 (Vs-), U?.4 (Vs-)
- net MOSFET-OUT: now also R?.1, R?.1, R?.2
- net at R?.2, R?.2: now also U?.3 (Vin+)
- net at R?.2: now also R?.1, U?.2 (Vin-)
- net +5V renamed +9V
- net +9V: now also R?.2, U?.7 (Vs+)
- new net: U?.3 (Vin+), U?.6 (Vout)
- new net: U?.2 (Vin-), U?.6 (Vout)
- new net: C?.2, R?.2, U?.7 (Vs+)
Other:
- note added: "Amplifier stage converts \nthe current output of the DAC \nto +5.25V +- 0.75V\n-> 4.5-6V"
- note added: "Optional follower Opamp\nto increase current output \nof the amplifier stage from \n250mA to 500mA max"
- note removed: "+5.25V +- 0.75V\n-> 4.5-6V"
- moved on the sheet: C?, R?, U?

Commit message: added dissipation Mosfet, cleaned up Main sheet
Other:
- note added: "Amplifier stage converts \nthe current output of the DAC \nto +5.25V +- 0.75V\n-> 4.5-6V\n(MOSFET \nIRFP4568)"
- note removed: "Amplifier stage converts \nthe current output of the DAC \nto +5.25V +- 0.75V\n-> 4.5-6V"
- moved on the sheet: C?, R?

Commit message: cleaned up power supplies
Changed lines of the file:
@@
 	3750 4200 4400 4200
 Wire Wire Line
-	3650 2050 3650 1850
-Wire Wire Line
-	3750 2050 3750 1850
-Wire Wire Line
-	3750 1850 3700 1850
+	3650 2050 3650 1650
+Wire Wire Line
+	3750 2050 3750 1650
+Wire Wire Line
+	3750 1650 3700 1650
 $Comp
 L Device:R R?
@@
 $EndComp
 Wire Wire Line
-	9200 1600 9200 1900
+	9200 1600 9200 1700
 $Comp
 L Device:R R?
@@
 L power:+3.3V #PWR?
 U 1 1 5D1B0B7D
-P 3700 1850
-F 0 "#PWR?" H 3700 1700 50  0001 C CNN
-F 1 "+3.3V" H 3715 2023 50  0000 C CNN
-F 2 "" H 3700 1850 50  0001 C CNN
-F 3 "" H 3700 1850 50  0001 C CNN
-	1    3700 1850
-	1    0    0    -1
-$EndComp
-Connection ~ 3700 1850
-Wire Wire Line
-	3700 1850 3650 1850
+P 3700 1650
+F 0 "#PWR?" H 3700 1500 50  0001 C CNN
+F 1 "+3.3V" H 3715 1823 50  0000 C CNN
+F 2 "" H 3700 1650 50  0001 C CNN
+F 3 "" H 3700 1650 50  0001 C CNN
+	1    3700 1650
+	1    0    0    -1
+$EndComp
+Wire Wire Line
+	3700 1650 3650 1650
 Wire Wire Line
 	4350 3050 4800 3050
@@
 Connection ~ 8100 2400
 Wire Wire Line
-	8100 2400 8100 1850
+	8100 2400 8100 1950
 $Comp
 L power:+9V #PWR?
@@
 	1    0    0    -1
 $EndComp
+Text GLabel 8200 1950 2    50   Input ~ 0
++9V
+Wire Wire Line
+	8200 1950 8100 1950
+Connection ~ 8100 1950
+Wire Wire Line
+	8100 1950 8100 1850
+Text GLabel 9300 1700 2    50   Input ~ 0
++12V
+Wire Wire Line
+	9300 1700 9200 1700
+Connection ~ 9200 1700
+Wire Wire Line
+	9200 1700 9200 1900
+Text GLabel 3850 1650 2    50   Input ~ 0
++3.3V
+Connection ~ 3700 1650
+Wire Wire Line
+	3750 1650 3850 1650
+Connection ~ 3750 1650
+Text GLabel 3550 4200 0    50   Input ~ 0
+GND
+Wire Wire Line
+	3550 4200 3650 4200
+Connection ~ 3650 4200
 $EndSCHEMATC

Commit message: error check on schematic done
Parts:
- gave numbers to parts that had none: 20
Changed lines of the file:
@@
 P 3750 3050
 AR Path="/5D0D129D" Ref="U?"  Part="1"
-AR Path="/5D0C0D63/5D0D129D" Ref="U?"  Part="1"
-F 0 "U?" H 3750 4231 50  0000 C CNN
+AR Path="/5D0C0D63/5D0D129D" Ref="U4"  Part="1"
+F 0 "U4" H 3750 4231 50  0000 C CNN
 F 1 "AD9744" H 3750 4140 50  0000 C CNN
 F 2 "Package_SO:TSSOP-28_4.4x9.7mm_P0.65mm" H 4350 3250 50  0001 C CNN
@@
 P 4500 4200
 AR Path="/5D0D12A3" Ref="#PWR?"  Part="1"
-AR Path="/5D0C0D63/5D0D12A3" Ref="#PWR?"  Part="1"
-F 0 "#PWR?" H 4500 3950 50  0001 C CNN
+AR Path="/5D0C0D63/5D0D12A3" Ref="#PWR013"  Part="1"
+F 0 "#PWR013" H 4500 3950 50  0001 C CNN
 F 1 "GND" H 4505 4027 50  0000 C CNN
 F 2 "" H 4500 4200 50  0001 C CNN
@@
 P 4700 3700
 AR Path="/5D0D12AB" Ref="C?"  Part="1"
-AR Path="/5D0C0D63/5D0D12AB" Ref="C?"  Part="1"
-F 0 "C?" H 4585 3654 50  0000 R CNN
+AR Path="/5D0C0D63/5D0D12AB" Ref="C17"  Part="1"
+F 0 "C17" H 4585 3654 50  0000 R CNN
 F 1 "100nF" H 4585 3745 50  0000 R CNN
 F 2 "" H 4738 3550 50  0001 C CNN
@@
 P 4400 3300
 AR Path="/5D0D12BB" Ref="R?"  Part="1"
-AR Path="/5D0C0D63/5D0D12BB" Ref="R?"  Part="1"
-F 0 "R?" H 4330 3254 50  0000 R CNN
+AR Path="/5D0C0D63/5D0D12BB" Ref="R10"  Part="1"
+F 0 "R10" H 4330 3254 50  0000 R CNN
 F 1 "3.84k" H 4330 3345 50  0000 R CNN
 F 2 "" V 4330 3300 50  0001 C CNN
@@
 	6200 2400 6500 2400
 $Comp
-L Device:R R?
+L Device:R R12
 U 1 1 5D15C614
 P 5450 3450
-F 0 "R?" H 5380 3404 50  0000 R CNN
+F 0 "R12" H 5380 3404 50  0000 R CNN
 F 1 "25R" H 5380 3495 50  0000 R CNN
 F 2 "" V 5380 3450 50  0001 C CNN
@@
 	4550 2950 5150 2950
 $Comp
-L Device:R R?
+L Device:R R13
 U 1 1 5D159343
 P 6050 2400
-F 0 "R?" V 6257 2400 50  0000 C CNN
+F 0 "R13" V 6257 2400 50  0000 C CNN
 F 1 "500R" V 6166 2400 50  0000 C CNN
 F 2 "" V 5980 2400 50  0001 C CNN
@@
 $EndComp
 $Comp
-L Device:R R?
+L Device:R R14
 U 1 1 5D160C2E
 P 6050 2950
-F 0 "R?" V 6257 2950 50  0000 C CNN
+F 0 "R14" V 6257 2950 50  0000 C CNN
 F 1 "500R" V 6166 2950 50  0000 C CNN
 F 2 "" V 5980 2950 50  0001 C CNN
@@
 $EndComp
 $Comp
-L Device:R R?
+L Device:R R11
 U 1 1 5D1624DF
 P 5150 3450
-F 0 "R?" H 5080 3404 50  0000 R CNN
+F 0 "R11" H 5080 3404 50  0000 R CNN
 F 1 "25R" H 5080 3495 50  0000 R CNN
 F 2 "" V 5080 3450 50  0001 C CNN
@@
 P 5600 2650
 AR Path="/5D164FAD" Ref="C?"  Part="1"
-AR Path="/5D0C0D63/5D164FAD" Ref="C?"  Part="1"
-F 0 "C?" H 5485 2604 50  0000 R CNN
+AR Path="/5D0C0D63/5D164FAD" Ref="C18"  Part="1"
+F 0 "C18" H 5485 2604 50  0000 R CNN
 F 1 "DNM" H 5485 2695 50  0000 R CNN
 F 2 "" H 5638 2500 50  0001 C CNN
@@
 P 8100 2750
 AR Path="/5D17131C" Ref="C?"  Part="1"
-AR Path="/5D0C0D63/5D17131C" Ref="C?"  Part="1"
-F 0 "C?" H 7985 2704 50  0000 R CNN
+AR Path="/5D0C0D63/5D17131C" Ref="C20"  Part="1"
+F 0 "C20" H 7985 2704 50  0000 R CNN
 F 1 "100nF" H 7985 2795 50  0000 R CNN
 F 2 "" H 8138 2600 50  0001 C CNN
@@
 Connection ~ 8100 4200
 $Comp
-L Reference_Voltage:LM285M-ADJ U?
+L Reference_Voltage:LM285M-ADJ U7
 U 1 1 5D17B099
 P 9200 2650
-F 0 "U?" V 9246 2562 50  0000 R CNN
+F 0 "U7" V 9246 2562 50  0000 R CNN
 F 1 "LM285M-ADJ" V 9155 2562 50  0000 R CNN
 F 2 "Package_SO:SOIC-8_3.9x4.9mm_P1.27mm" H 9200 2450 50  0001 C CIN
@@
 	9200 1600 9200 1700
 $Comp
-L Device:R R?
+L Device:R R21
 U 1 1 5D17E776
 P 9200 2050
-F 0 "R?" H 9270 2096 50  0000 L CNN
+F 0 "R21" H 9270 2096 50  0000 L CNN
 F 1 "50k" H 9270 2005 50  0000 L CNN
 F 2 "" V 9130 2050 50  0001 C CNN
@@
 $EndComp
 $Comp
-L Device:R R?
+L Device:R R19
 U 1 1 5D185936
 P 8800 2450
-F 0 "R?" H 8870 2496 50  0000 L CNN
+F 0 "R19" H 8870 2496 50  0000 L CNN
 F 1 "130k" H 8870 2405 50  0000 L CNN
 F 2 "" V 8730 2450 50  0001 C CNN
@@
 	9200 2500 9200 2300
 $Comp
-L Device:R R?
+L Device:R R20
 U 1 1 5D1853A4
 P 8800 2850
-F 0 "R?" H 8870 2896 50  0000 L CNN
+F 0 "R20" H 8870 2896 50  0000 L CNN
 F 1 "422k" H 8870 2805 50  0000 L CNN
 F 2 "" V 8730 2850 50  0001 C CNN
@@
 Vout = 5.25V
 $Comp
-L Device:R R?
+L Device:R R18
 U 1 1 5D1A8AA6
 P 8550 2650
-F 0 "R?" H 8620 2696 50  0000 L CNN
+F 0 "R18" H 8620 2696 50  0000 L CNN
 F 1 "1k" H 8620 2605 50  0000 L CNN
 F 2 "" V 8480 2650 50  0001 C CNN
@@
 Amplifier stage converts \nthe current output of the DAC \nto +5.25V +- 0.75V\n-> 4.5-6V\n(MOSFET \nIRFP4568)
 $Comp
-L power:+3.3V #PWR?
+L power:+3.3V #PWR012
 U 1 1 5D1B0B7D
 P 3700 1650
-F 0 "#PWR?" H 3700 1500 50  0001 C CNN
+F 0 "#PWR012" H 3700 1500 50  0001 C CNN
 F 1 "+3.3V" H 3715 1823 50  0000 C CNN
 F 2 "" H 3700 1650 50  0001 C CNN
@@
 MOSFET-OUT
 $Comp
-L OS-LD:THS3091 U?
+L OS-LD:THS3091 U5
 U 1 1 5D08DF18
 P 7000 2450
-F 0 "U?" H 7000 2825 50  0000 C CNN
+F 0 "U5" H 7000 2825 50  0000 C CNN
 F 1 "THS3091" H 7000 2734 50  0000 C CNN
 F 2 "" H 6950 2400 50  0001 C CNN
@@
 	8100 2400 8100 1950
 $Comp
-L power:+9V #PWR?
+L power:+9V #PWR014
 U 1 1 5D09D7FB
 P 8100 1850
-F 0 "#PWR?" H 8100 1700 50  0001 C CNN
+F 0 "#PWR014" H 8100 1700 50  0001 C CNN
 F 1 "+9V" H 8115 2023 50  0000 C CNN
 F 2 "" H 8100 1850 50  0001 C CNN
@@
 $EndComp
 $Comp
-L Device:R R?
+L Device:R R15
 U 1 1 5D0A1BBC
 P 7200 1900
-F 0 "R?" V 7407 1900 50  0000 C CNN
+F 0 "R15" V 7407 1900 50  0000 C CNN
 F 1 "750R" V 7316 1900 50  0000 C CNN
 F 2 "" V 7130 1900 50  0001 C CNN
@@
 	7500 2500 7350 2500
 $Comp
-L OS-LD:THS3091 U?
+L OS-LD:THS3091 U6
 U 1 1 5D0AA5C9
 P 7050 3500
-F 0 "U?" H 7050 3875 50  0000 C CNN
+F 0 "U6" H 7050 3875 50  0000 C CNN
 F 1 "THS3091" H 7050 3784 50  0000 C CNN
 F 2 "" H 7000 3450 50  0001 C CNN
@@
 P 7750 3600
 AR Path="/5D0C651A" Ref="C?"  Part="1"
-AR Path="/5D0C0D63/5D0C651A" Ref="C?"  Part="1"
-F 0 "C?" H 7635 3554 50  0000 R CNN
+AR Path="/5D0C0D63/5D0C651A" Ref="C19"  Part="1"
+F 0 "C19" H 7635 3554 50  0000 R CNN
 F 1 "100nF" H 7635 3645 50  0000 R CNN
 F 2 "" H 7788 3450 50  0001 C CNN
@@
 	7500 2800 7500 2500
 $Comp
-L Device:R R?
+L Device:R R16
 U 1 1 5D0D5F3D
 P 7500 2150
-F 0 "R?" V 7707 2150 50  0000 C CNN
+F 0 "R16" V 7707 2150 50  0000 C CNN
 F 1 "25R" V 7616 2150 50  0000 C CNN
 F 2 "" V 7430 2150 50  0001 C CNN
@@
 	7500 2400 8100 2400
 $Comp
-L Device:R R?
+L Device:R R17
 U 1 1 5D0DB2E7
 P 7750 2600
-F 0 "R?" V 7957 2600 50  0000 C CNN
+F 0 "R17" V 7957 2600 50  0000 C CNN
 F 1 "25R" V 7866 2600 50  0000 C CNN
 F 2 "" V 7680 2600 50  0001 C CNN
@@
 	7350 1900 7500 1900
 $Comp
-L power:+12V #PWR?
+L power:+12V #PWR015
 U 1 1 5D17CC85
 P 9200 1600
-F 0 "#PWR?" H 9200 1450 50  0001 C CNN
+F 0 "#PWR015" H 9200 1450 50  0001 C CNN
 F 1 "+12V" H 9215 1773 50  0000 C CNN
 F 2 "" H 9200 1600 50  0001 C CNN
