File: Hardware/Output.sch (KiCad schematic (older format))
At the start: 20 parts, among them U4 AD9744, U5 THS3091, U6 THS3091, U7 LM285M-ADJ

Commit message: removed labels from power connections. powr conn already global
Changed lines of the file:
@@
 AR Path="/5D0D129D" Ref="U?"  Part="1"
 AR Path="/5D0C0D63/5D0D129D" Ref="U4"  Part="1"
-F 0 "U4" H 3750 4231 50  0000 C CNN
-F 1 "AD9744" H 3750 4140 50  0000 C CNN
+F 0 "U4" H 4000 4100 50  0000 C CNN
+F 1 "AD9744" H 4100 4000 50  0000 C CNN
 F 2 "Package_SO:TSSOP-28_4.4x9.7mm_P0.65mm" H 4350 3250 50  0001 C CNN
 F 3 "https://www.analog.com/media/en/technical-documentation/data-sheets/AD9744.pdf" H 4350 3250 50  0001 C CNN
@@
 	0    -1   -1   0
 $EndComp
-Wire Wire Line
-	9200 1600 9200 1700
 $Comp
 L Device:R R21
@@
 	7350 2400 7500 2400
 Connection ~ 8100 2400
-Wire Wire Line
-	8100 2400 8100 1950
 $Comp
 L power:+9V #PWR014
@@
 	1    0    0    -1
 $EndComp
-Text GLabel 8200 1950 2    50   Input ~ 0
-+9V
-Wire Wire Line
-	8200 1950 8100 1950
-Connection ~ 8100 1950
-Wire Wire Line
-	8100 1950 8100 1850
-Text GLabel 9300 1700 2    50   Input ~ 0
-+12V
-Wire Wire Line
-	9300 1700 9200 1700
-Connection ~ 9200 1700
-Wire Wire Line
-	9200 1700 9200 1900
-Text GLabel 3850 1650 2    50   Input ~ 0
-+3.3V
 Connection ~ 3700 1650
 Wire Wire Line
-	3750 1650 3850 1650
-Connection ~ 3750 1650
-Text GLabel 3550 4200 0    50   Input ~ 0
-GND
-Wire Wire Line
-	3550 4200 3650 4200
-Connection ~ 3650 4200
+	9200 1600 9200 1900
+Wire Wire Line
+	8100 1850 8100 2400
 $EndSCHEMATC

Commit message: fixed output amp biasing
Parts:
- removed R16: 25R, Resistor_SMD:R_0603_1608Metric, symbol Device:R
Connections:
- net +9V: now also C19.2, U6.7 (Vs+)
- net MOSFET-OUT: now also U6.2 (Vin-), U6.6 (Vout); no longer R15.2, R17.1
- net at R14.2, U5.3 (Vin+): now also R18.1; no longer R18.2
- net at U5.6 (Vout), U6.3 (Vin+): now also R15.2
- net at R19.1, R21.2, U7.8 (K): now also R18.2; no longer R18.1
- now unconnected: R17.2
Other:
- moved on the sheet: C17, C18, C19, C20, R10, R11, R12, R13, R14, R15, R17, R18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

Commit message: removed redundant resistor
Parts:
- removed R17: 25R, Resistor_SMD:R_0603_1608Metric, symbol Device:R
Changed lines of the file:
@@
 	-1   0    0    1
-$EndComp
-$Comp
-L Device:R R17
-U 1 1 5D0DB2E7
-P 5300 5350
-F 0 "R17" V 5507 5350 50  0000 C CNN
-F 1 "25R" V 5416 5350 50  0000 C CNN
-F 2 "Resistor_SMD:R_0603_1608Metric" V 5230 5350 50  0001 C CNN
-F 3 "~" H 5300 5350 50  0001 C CNN
-	1    5300 5350
-	1    0    0    -1
 $EndComp
 Text Notes 7600 3450 0    50   ~ 0

Commit message: added footprints to components
Parts:
- C18: footprint (none) -> Capacitor_SMD:C_0603_1608Metric
- U5, U6: footprint (none) -> Package_SO:SOIC-8_3.9x4.9mm_P1.27mm
Changed lines of the file:
@@
 F 0 "C18" H 4335 3004 50  0000 R CNN
 F 1 "DNM" H 4335 3095 50  0000 R CNN
-F 2 "" H 4488 2900 50  0001 C CNN
+F 2 "Capacitor_SMD:C_0603_1608Metric" H 4488 2900 50  0001 C CNN
 F 3 "~" H 4450 3050 50  0001 C CNN
 	1    4450 3050
@@
 F 0 "U5" H 5850 3225 50  0000 C CNN
 F 1 "THS3091" H 5850 3134 50  0000 C CNN
-F 2 "" H 5800 2800 50  0001 C CNN
+F 2 "Package_SO:SOIC-8_3.9x4.9mm_P1.27mm" H 5800 2800 50  0001 C CNN
 F 3 "" H 5800 2800 50  0001 C CNN
 	1    5850 2850
@@
 F 0 "U6" H 8050 3225 50  0000 C CNN
 F 1 "THS3091" H 8050 3134 50  0000 C CNN
-F 2 "" H 8000 2800 50  0001 C CNN
+F 2 "Package_SO:SOIC-8_3.9x4.9mm_P1.27mm" H 8000 2800 50  0001 C CNN
 F 3 "" H 8000 2800 50  0001 C CNN
 	1    8050 2850

Commit message: finished placement. started routing
Parts:
- added C7, C8: 100nF, Capacitor_SMD:C_0603_1608Metric, symbol Device:C
Connections:
- net +3V3: now also C7.2, C8.2
- net GND: now also C7.1, C8.1
Changed lines of the file:
@@
 AR Path="/5D0D129D" Ref="U?"  Part="1"
 AR Path="/5D0C0D63/5D0D129D" Ref="U4"  Part="1"
-F 0 "U4" H 2850 4500 50  0000 C CNN
-F 1 "AD9744" H 2950 4400 50  0000 C CNN
+F 0 "U4" H 2950 4400 50  0000 C CNN
+F 1 "AD9744" H 2200 4400 50  0000 C CNN
 F 2 "Package_SO:TSSOP-28_4.4x9.7mm_P0.65mm" H 3200 3650 50  0001 C CNN
 F 3 "https://www.analog.com/media/en/technical-documentation/data-sheets/AD9744.pdf" H 3200 3650 50  0001 C CNN
@@
 Wire Wire Line
 	2600 4600 3250 4600
-Wire Wire Line
-	2500 2450 2500 2050
-Wire Wire Line
-	2600 2450 2600 2050
-Wire Wire Line
-	2600 2050 2550 2050
 $Comp
 L Device:R R?
@@
 L power:+3.3V #PWR012
 U 1 1 5D1B0B7D
-P 2550 2050
-F 0 "#PWR012" H 2550 1900 50  0001 C CNN
-F 1 "+3.3V" H 2565 2223 50  0000 C CNN
-F 2 "" H 2550 2050 50  0001 C CNN
-F 3 "" H 2550 2050 50  0001 C CNN
-	1    2550 2050
-	1    0    0    -1
-$EndComp
-Wire Wire Line
-	2550 2050 2500 2050
+P 2600 1900
+F 0 "#PWR012" H 2600 1750 50  0001 C CNN
+F 1 "+3.3V" H 2615 2073 50  0000 C CNN
+F 2 "" H 2600 1900 50  0001 C CNN
+F 3 "" H 2600 1900 50  0001 C CNN
+	1    2600 1900
+	1    0    0    -1
+$EndComp
 Wire Wire Line
 	3200 3450 3650 3450
@@
 Wire Notes Line
 	4750 2000 4750 3450
-Connection ~ 2550 2050
 Wire Wire Line
 	8400 2800 8750 2800
@@
 	9500 2900 8500 2900
 Connection ~ 8500 2900
+$Comp
+L Device:C C?
+U 1 1 60145D90
+P 2850 2050
+AR Path="/60145D90" Ref="C?"  Part="1"
+AR Path="/5D0C0D63/60145D90" Ref="C8"  Part="1"
+F 0 "C8" H 2735 2004 50  0000 R CNN
+F 1 "100nF" H 2735 2095 50  0000 R CNN
+F 2 "Capacitor_SMD:C_0603_1608Metric" H 2888 1900 50  0001 C CNN
+F 3 "~" H 2850 2050 50  0001 C CNN
+	1    2850 2050
+	-1   0    0    1
+$EndComp
+$Comp
+L Device:C C?
+U 1 1 60147488
+P 2100 2050
+AR Path="/60147488" Ref="C?"  Part="1"
+AR Path="/5D0C0D63/60147488" Ref="C7"  Part="1"
+F 0 "C7" H 1985 2004 50  0000 R CNN
+F 1 "100nF" H 1985 2095 50  0000 R CNN
+F 2 "Capacitor_SMD:C_0603_1608Metric" H 2138 1900 50  0001 C CNN
+F 3 "~" H 2100 2050 50  0001 C CNN
+	1    2100 2050
+	-1   0    0    1
+$EndComp
+Wire Wire Line
+	2600 1900 2850 1900
+Wire Wire Line
+	2600 1900 2600 2300
+Connection ~ 2600 1900
+Wire Wire Line
+	2100 1900 2600 1900
+Wire Wire Line
+	2600 2300 2500 2300
+Wire Wire Line
+	2500 2300 2500 2450
+Connection ~ 2600 2300
+Wire Wire Line
+	2600 2300 2600 2450
+$Comp
+L power:GND #PWR?
+U 1 1 60151AD5
+P 2100 2200
+AR Path="/60151AD5" Ref="#PWR?"  Part="1"
+AR Path="/5D0C0D63/60151AD5" Ref="#PWR055"  Part="1"
+F 0 "#PWR055" H 2100 1950 50  0001 C CNN
+F 1 "GND" H 2105 2027 50  0000 C CNN
+F 2 "" H 2100 2200 50  0001 C CNN
+F 3 "" H 2100 2200 50  0001 C CNN
+	1    2100 2200
+	1    0    0    -1
+$EndComp
+$Comp
+L power:GND #PWR?
+U 1 1 6015229A
+P 2850 2200
+AR Path="/6015229A" Ref="#PWR?"  Part="1"
+AR Path="/5D0C0D63/6015229A" Ref="#PWR056"  Part="1"
+F 0 "#PWR056" H 2850 1950 50  0001 C CNN
+F 1 "GND" H 3000 2150 50  0000 C CNN
+F 2 "" H 2850 2200 50  0001 C CNN
+F 3 "" H 2850 2200 50  0001 C CNN
+	1    2850 2200
+	1    0    0    -1
+$EndComp
 $EndSCHEMATC
