File: Hardware/Power.sch (KiCad schematic (older format))
At the start: 38 parts, among them J6 Barrel_Jack_MountingPin, U10 LM2734Y, U8 LM2734Y

Commit message: fixed file name. used kicad default gitignore
Parts:
- gave numbers to parts that had none: 16
Changed lines of the file:
@@
 	10450 2750 10450 2550
 $Comp
-L TPS63700:TPS63700DRCT U?
+L TPS63700:TPS63700DRCT U9
 U 1 1 5F63BF1B
 P 2550 5200
-F 0 "U?" H 3150 5387 60  0000 C CNN
+F 0 "U9" H 3150 5387 60  0000 C CNN
 F 1 "TPS63700DRCT" H 3150 5281 60  0000 C CNN
 F 2 "DRC10_2P4X1P65" H 3150 5240 60  0001 C CNN
@@
 	4050 6000 4600 6000
 $Comp
-L Device:R R?
+L Device:R R36
 U 1 1 5F63FB14
 P 4600 5350
-F 0 "R?" H 4670 5396 50  0000 L CNN
+F 0 "R36" H 4670 5396 50  0000 L CNN
 F 1 "150k" H 4650 5350 50  0000 L CNN
 F 2 "" V 4530 5350 50  0001 C CNN
@@
 $EndComp
 $Comp
-L Device:R R?
+L Device:R R38
 U 1 1 5F640A27
 P 4600 5800
-F 0 "R?" H 4670 5846 50  0000 L CNN
+F 0 "R38" H 4670 5846 50  0000 L CNN
 F 1 "410k" H 4670 5755 50  0000 L CNN
 F 2 "" V 4530 5800 50  0001 C CNN
@@
 $EndComp
 $Comp
-L Device:R R?
+L Device:R R39
 U 1 1 5F64149F
 P 5050 5800
-F 0 "R?" H 5120 5846 50  0000 L CNN
+F 0 "R39" H 5120 5846 50  0000 L CNN
 F 1 "100k" H 5120 5755 50  0000 L CNN
 F 2 "" V 4980 5800 50  0001 C CNN
@@
 $EndComp
 $Comp
-L Device:C_Small C?
+L Device:C_Small C2
 U 1 1 5F642E45
 P 4150 5200
-F 0 "C?" H 4242 5246 50  0000 L CNN
+F 0 "C2" H 4242 5246 50  0000 L CNN
 F 1 "0.22uF" H 4242 5155 50  0000 L CNN
 F 2 "" H 4150 5200 50  0001 C CNN
@@
 $EndComp
 $Comp
-L power:-3V3 #PWR?
+L power:-3V3 #PWR0114
 U 1 1 5F63CC11
 P 6150 6000
-F 0 "#PWR?" H 6150 6100 50  0001 C CNN
+F 0 "#PWR0114" H 6150 6100 50  0001 C CNN
 F 1 "-3V3" H 6165 6173 50  0000 C CNN
 F 2 "" H 6150 6000 50  0001 C CNN
@@
 	5050 6000 5250 6000
 $Comp
-L Device:C_Small C?
+L Device:C_Small C4
 U 1 1 5F662B7D
 P 4850 5600
-F 0 "C?" V 4750 5650 50  0000 C CNN
+F 0 "C4" V 4750 5650 50  0000 C CNN
 F 1 "10pF" V 4950 5650 50  0000 C CNN
 F 2 "" H 4850 5600 50  0001 C CNN
@@
 	5050 5600 5050 5650
 $Comp
-L Device:C_Small C?
+L Device:C_Small C6
 U 1 1 5F669437
 P 5250 6150
-F 0 "C?" V 5300 6200 50  0000 L CNN
+F 0 "C6" V 5300 6200 50  0000 L CNN
 F 1 "4.7uF" V 5150 6000 50  0000 L CNN
 F 2 "" H 5250 6150 50  0001 C CNN
@@
 $EndComp
 $Comp
-L Device:C_Small C?
+L Device:C_Small C7
 U 1 1 5F669C76
 P 5500 6150
-F 0 "C?" V 5550 6200 50  0000 L CNN
+F 0 "C7" V 5550 6200 50  0000 L CNN
 F 1 "4.7uF" V 5400 6000 50  0000 L CNN
 F 2 "" H 5500 6150 50  0001 C CNN
@@
 $EndComp
 $Comp
-L Device:C_Small C?
+L Device:C_Small C8
 U 1 1 5F669E13
 P 5750 6150
-F 0 "C?" V 5800 6200 50  0000 L CNN
+F 0 "C8" V 5800 6200 50  0000 L CNN
 F 1 "4.7uF" V 5650 6000 50  0000 L CNN
 F 2 "" H 5750 6150 50  0001 C CNN
@@
 $EndComp
 $Comp
-L Device:C_Small C?
+L Device:C_Small C9
 U 1 1 5F66A15D
 P 6000 6150
-F 0 "C?" V 6050 6200 50  0000 L CNN
+F 0 "C9" V 6050 6200 50  0000 L CNN
 F 1 "4.7uF" V 5900 6000 50  0000 L CNN
 F 2 "" H 6000 6150 50  0001 C CNN
@@
 	6000 6000 6150 6000
 $Comp
-L power:GND #PWR?
+L power:GND #PWR0115
 U 1 1 5F67739A
 P 6150 6350
-F 0 "#PWR?" H 6150 6100 50  0001 C CNN
+F 0 "#PWR0115" H 6150 6100 50  0001 C CNN
 F 1 "GND" H 6155 6177 50  0000 C CNN
 F 2 "" H 6150 6350 50  0001 C CNN
@@
 	6000 6350 6150 6350
 $Comp
-L power:GND #PWR?
+L power:GND #PWR0116
 U 1 1 5F686EBA
 P 4200 6550
-F 0 "#PWR?" H 4200 6300 50  0001 C CNN
+F 0 "#PWR0116" H 4200 6300 50  0001 C CNN
 F 1 "GND" H 4205 6377 50  0000 C CNN
 F 2 "" H 4200 6550 50  0001 C CNN
@@
 $EndComp
 $Comp
-L Device:L L?
+L Device:L L3
 U 1 1 5F687B61
 P 4200 6400
-F 0 "L?" H 4253 6446 50  0000 L CNN
+F 0 "L3" H 4253 6446 50  0000 L CNN
 F 1 "L" H 4253 6355 50  0000 L CNN
 F 2 "" H 4200 6400 50  0001 C CNN
@@
 $EndComp
 $Comp
-L Device:D_Schottky D?
+L Device:D_Schottky D7
 U 1 1 5F68AC87
 P 4650 6250
-F 0 "D?" H 4650 6350 50  0000 C CNN
+F 0 "D7" H 4650 6350 50  0000 C CNN
 F 1 "SL03-GS08" H 4650 6150 50  0000 C CNN
 F 2 "" H 4650 6250 50  0001 C CNN
@@
 	5050 6250 5050 6000
 $Comp
-L power:GND #PWR?
+L power:GND #PWR0117
 U 1 1 5F694AC5
 P 4150 5300
-F 0 "#PWR?" H 4150 5050 50  0001 C CNN
+F 0 "#PWR0117" H 4150 5050 50  0001 C CNN
 F 1 "GND" H 4155 5127 50  0000 C CNN
 F 2 "" H 4150 5300 50  0001 C CNN
@@
 $EndComp
 $Comp
-L power:GND #PWR?
+L power:GND #PWR0118
 U 1 1 5F694EE7
 P 2150 6300
-F 0 "#PWR?" H 2150 6050 50  0001 C CNN
+F 0 "#PWR0118" H 2150 6050 50  0001 C CNN
 F 1 "GND" H 2155 6127 50  0000 C CNN
 F 2 "" H 2150 6300 50  0001 C CNN
@@
 $EndComp
 $Comp
-L Device:C_Small C?
+L Device:C_Small C10
 U 1 1 5F695350
 P 1800 6200
-F 0 "C?" H 1708 6154 50  0000 R CNN
+F 0 "C10" H 1708 6154 50  0000 R CNN
 F 1 "4.7nF" H 1708 6245 50  0000 R CNN
 F 2 "" H 1800 6200 50  0001 C CNN
@@
 $EndComp
 $Comp
-L power:GND #PWR?
+L power:GND #PWR0119
 U 1 1 5F696088
 P 1800 6300
-F 0 "#PWR?" H 1800 6050 50  0001 C CNN
+F 0 "#PWR0119" H 1800 6050 50  0001 C CNN
 F 1 "GND" H 1805 6127 50  0000 C CNN
 F 2 "" H 1800 6300 50  0001 C CNN
@@
 $EndComp
 $Comp
-L Device:C_Small C?
+L Device:C_Small C5
 U 1 1 5F6962C6
 P 1400 5850
-F 0 "C?" H 1308 5804 50  0000 R CNN
+F 0 "C5" H 1308 5804 50  0000 R CNN
 F 1 "10uF" H 1308 5895 50  0000 R CNN
 F 2 "" H 1400 5850 50  0001 C CNN
@@
 $EndComp
 $Comp
-L power:GND #PWR?
+L power:GND #PWR0120
 U 1 1 5F69679F
 P 1400 6300
-F 0 "#PWR?" H 1400 6050 50  0001 C CNN
+F 0 "#PWR0120" H 1400 6050 50  0001 C CNN
 F 1 "GND" H 1405 6127 50  0000 C CNN
 F 2 "" H 1400 6300 50  0001 C CNN
@@
 Connection ~ 2250 5350
 $Comp
-L Device:C_Small C?
+L Device:C_Small C3
 U 1 1 5F6D20D3
 P 1900 5450
-F 0 "C?" H 1808 5404 50  0000 R CNN
+F 0 "C3" H 1808 5404 50  0000 R CNN
 F 1 "0.1uF" H 1808 5495 50  0000 R CNN
 F 2 "" H 1900 5450 50  0001 C CNN
@@
 	1900 5350 2250 5350
 $Comp
-L power:GND #PWR?
+L power:GND #PWR0121
 U 1 1 5F6D24D5
 P 1900 5550
-F 0 "#PWR?" H 1900 5300 50  0001 C CNN
+F 0 "#PWR0121" H 1900 5300 50  0001 C CNN
 F 1 "GND" H 1905 5377 50  0000 C CNN
 F 2 "" H 1900 5550 50  0001 C CNN
@@
 	1600 5650 1600 5700
 $Comp
-L Device:R R?
+L Device:R R37
 U 1 1 5F6BAA22
 P 1600 5500
-F 0 "R?" H 1670 5546 50  0000 L CNN
+F 0 "R37" H 1670 5546 50  0000 L CNN
 F 1 "10R" H 1670 5455 50  0000 L CNN
 F 2 "" V 1530 5500 50  0001 C CNN

Commit message: removed labels from power connections. powr conn already global
Other:
- moved on the sheet: C25, C26, C27, D3, D4, D5, L2, R25, R26, R27, U10

Commit message: fixed resistor values for the 9V supply
Parts:
- C25: value 10uF -> 10uF 25V
- C26: value 10nF -> 10nF 16V
- C27: value 22uF -> 22uF 16V
- L2: value SLF7032T-6R8M1R -> 22uH 1.4 A; MPN (none) -> SLF7045T-220M1R3-1PF
- R25: value 10k -> 100k
- R26: value 10k -> 102k 1%
- R27: value 10k -> 10.2k 1%
Connections:
- no-connect marks 0 -> 1
Other:
- moved on the sheet: C25, R25
Changed lines of the file:
@@
 L power:+12V #PWR016
 U 1 1 5D13CAC2
-P 2150 2350
-F 0 "#PWR016" H 2150 2200 50  0001 C CNN
-F 1 "+12V" H 2165 2523 50  0000 C CNN
-F 2 "" H 2150 2350 50  0001 C CNN
-F 3 "" H 2150 2350 50  0001 C CNN
-	1    2150 2350
+P 2150 2750
+F 0 "#PWR016" H 2150 2600 50  0001 C CNN
+F 1 "+12V" H 2165 2923 50  0000 C CNN
+F 2 "" H 2150 2750 50  0001 C CNN
+F 3 "" H 2150 2750 50  0001 C CNN
+	1    2150 2750
 	1    0    0    -1
 $EndComp
@@
 L power:+5V #PWR018
 U 1 1 5D13D9BD
-P 5700 2550
-F 0 "#PWR018" H 5700 2400 50  0001 C CNN
-F 1 "+5V" H 5715 2723 50  0000 C CNN
-F 2 "" H 5700 2550 50  0001 C CNN
-F 3 "" H 5700 2550 50  0001 C CNN
-	1    5700 2550
+P 5700 2700
+F 0 "#PWR018" H 5700 2550 50  0001 C CNN
+F 1 "+5V" H 5715 2873 50  0000 C CNN
+F 2 "" H 5700 2700 50  0001 C CNN
+F 3 "" H 5700 2700 50  0001 C CNN
+	1    5700 2700
 	1    0    0    -1
 $EndComp
@@
 L power:+12V #PWR020
 U 1 1 5D146985
-P 7100 2500
-F 0 "#PWR020" H 7100 2350 50  0001 C CNN
-F 1 "+12V" H 7115 2673 50  0000 C CNN
-F 2 "" H 7100 2500 50  0001 C CNN
-F 3 "" H 7100 2500 50  0001 C CNN
-	1    7100 2500
+P 6800 2650
+F 0 "#PWR020" H 6800 2500 50  0001 C CNN
+F 1 "+12V" H 6815 2823 50  0000 C CNN
+F 2 "" H 6800 2650 50  0001 C CNN
+F 3 "" H 6800 2650 50  0001 C CNN
+	1    6800 2650
 	1    0    0    -1
 $EndComp
@@
 L Device:R_Small R25
 U 1 1 5D146A1A
-P 7450 2800
-F 0 "R25" H 7509 2846 50  0000 L CNN
-F 1 "10k" H 7509 2755 50  0000 L CNN
-F 2 "Resistor_SMD:R_0603_1608Metric" H 7450 2800 50  0001 C CNN
-F 3 "~" H 7450 2800 50  0001 C CNN
-	1    7450 2800
-	1    0    0    -1
-$EndComp
-Wire Wire Line
-	7450 2900 7650 2900
+P 7150 2900
+F 0 "R25" H 7209 2946 50  0000 L CNN
+F 1 "100k" H 7209 2855 50  0000 L CNN
+F 2 "Resistor_SMD:R_0603_1608Metric" H 7150 2900 50  0001 C CNN
+F 3 "~" H 7150 2900 50  0001 C CNN
+	1    7150 2900
+	1    0    0    -1
+$EndComp
 $Comp
 L Device:C_Small C25
 U 1 1 5D147FA9
-P 7100 2800
-F 0 "C25" H 7192 2846 50  0000 L CNN
-F 1 "10uF" H 7192 2755 50  0000 L CNN
-F 2 "Capacitor_SMD:C_0603_1608Metric" H 7100 2800 50  0001 C CNN
-F 3 "~" H 7100 2800 50  0001 C CNN
-	1    7100 2800
+P 6800 2800
+F 0 "C25" H 6500 2900 50  0000 L CNN
+F 1 "10uF 25V" H 6350 2800 50  0000 L CNN
+F 2 "Capacitor_SMD:C_0603_1608Metric" H 6800 2800 50  0001 C CNN
+F 3 "~" H 6800 2800 50  0001 C CNN
+	1    6800 2800
 	1    0    0    -1
 $EndComp
@@
 U 1 1 5D152A1F
 P 9050 2800
-F 0 "L2" V 8872 2800 50  0000 C CNN
-F 1 "SLF7032T-6R8M1R" V 8950 3100 50  0000 C CNN
+F 0 "L2" V 8950 2800 50  0000 C CNN
+F 1 "22uH 1.4 A" V 9150 2900 50  0000 C CNN
 F 2 "Inductor_SMD:L_7.3x7.3_H3.5" H 9050 2800 50  0001 C CNN
 F 3 "~" H 9050 2800 50  0001 C CNN
+F 4 "SLF7045T-220M1R3-1PF" V 9050 2800 50  0001 C CNN "MPN"
 	1    9050 2800
 	0    1    1    0
 $EndComp
 Wire Wire Line
-	7100 2500 7100 2700
+	6800 2650 6800 2700
 $Comp
 L Device:C_Small C27
@@
 P 10300 3050
 F 0 "C27" H 10392 3096 50  0000 L CNN
-F 1 "22uF" H 10392 3005 50  0000 L CNN
+F 1 "22uF 16V" H 10392 3005 50  0000 L CNN
 F 2 "Capacitor_SMD:C_0603_1608Metric" H 10300 3050 50  0001 C CNN
 F 3 "~" H 10300 3050 50  0001 C CNN
@@
 	1    0    0    -1
 $EndComp
-Connection ~ 7100 2700
-Wire Wire Line
-	7100 2700 7450 2700
-Connection ~ 7450 2700
-Wire Wire Line
-	7450 2700 7650 2700
+Connection ~ 6800 2700
+Wire Wire Line
+	6800 2700 7150 2700
 $Comp
 L Device:R_Small R27
@@
 P 9850 3500
 F 0 "R27" H 9909 3546 50  0000 L CNN
-F 1 "10k" H 9909 3455 50  0000 L CNN
+F 1 "10.2k 1%" H 9909 3455 50  0000 L CNN
 F 2 "Resistor_SMD:R_0603_1608Metric" H 9850 3500 50  0001 C CNN
 F 3 "~" H 9850 3500 50  0001 C CNN
@@
 L power:+9V #PWR021
 U 1 1 5D1829E8
-P 10300 2600
-F 0 "#PWR021" H 10300 2450 50  0001 C CNN
-F 1 "+9V" H 10315 2773 50  0000 C CNN
-F 2 "" H 10300 2600 50  0001 C CNN
-F 3 "" H 10300 2600 50  0001 C CNN
-	1    10300 2600
+P 10300 2750
+F 0 "#PWR021" H 10300 2600 50  0001 C CNN
+F 1 "+9V" H 10315 2923 50  0000 C CNN
+F 2 "" H 10300 2750 50  0001 C CNN
+F 3 "" H 10300 2750 50  0001 C CNN
+	1    10300 2750
 	1    0    0    -1
 $EndComp
@@
 $EndComp
 Wire Wire Line
-	2150 2350 2150 2850
-Wire Wire Line
-	5700 2550 5700 2750
-$Comp
-L power:GND #PWR?
+	2150 2750 2150 2850
+Wire Wire Line
+	5700 2700 5700 2750
+$Comp
+L power:GND #PWR0122
 U 1 1 5FDFBB7D
-P 7100 3000
-F 0 "#PWR?" H 7100 2750 50  0001 C CNN
-F 1 "GND" H 7105 2827 50  0000 C CNN
-F 2 "" H 7100 3000 50  0001 C CNN
-F 3 "" H 7100 3000 50  0001 C CNN
-	1    7100 3000
-	1    0    0    -1
-$EndComp
-Wire Wire Line
-	7100 2900 7100 3000
-$Comp
-L power:GND #PWR?
+P 6800 3000
+F 0 "#PWR0122" H 6800 2750 50  0001 C CNN
+F 1 "GND" H 6805 2827 50  0000 C CNN
+F 2 "" H 6800 3000 50  0001 C CNN
+F 3 "" H 6800 3000 50  0001 C CNN
+	1    6800 3000
+	1    0    0    -1
+$EndComp
+Wire Wire Line
+	6800 2900 6800 3000
+$Comp
+L power:GND #PWR0123
 U 1 1 5FE0CC7B
 P 8050 3150
-F 0 "#PWR?" H 8050 2900 50  0001 C CNN
+F 0 "#PWR0123" H 8050 2900 50  0001 C CNN
 F 1 "GND" H 8055 2977 50  0000 C CNN
 F 2 "" H 8050 3150 50  0001 C CNN
@@
 	8050 3100 8050 3150
 $Comp
-L power:GND #PWR?
+L power:GND #PWR0124
 U 1 1 5FE120E8
 P 9850 3600
-F 0 "#PWR?" H 9850 3350 50  0001 C CNN
+F 0 "#PWR0124" H 9850 3350 50  0001 C CNN
 F 1 "GND" H 9855 3427 50  0000 C CNN
 F 2 "" H 9850 3600 50  0001 C CNN
@@
 P 9850 3200
 F 0 "R26" H 9909 3246 50  0000 L CNN
-F 1 "10k" H 9909 3155 50  0000 L CNN
+F 1 "102k 1%" H 9909 3155 50  0000 L CNN
 F 2 "Resistor_SMD:R_0603_1608Metric" H 9850 3200 50  0001 C CNN
 F 3 "~" H 9850 3200 50  0001 C CNN
@@
 $EndComp
 $Comp
-L power:GND #PWR?
+L power:GND #PWR0125
 U 1 1 5FE25ABE
 P 8700 3150
-F 0 "#PWR?" H 8700 2900 50  0001 C CNN
+F 0 "#PWR0125" H 8700 2900 50  0001 C CNN
 F 1 "GND" H 8700 3000 50  0000 C CNN
 F 2 "" H 8700 3150 50  0001 C CNN
@@
 $EndComp
 Wire Wire Line
-	10300 2600 10300 2800
+	10300 2750 10300 2800
 Wire Wire Line
 	10300 2800 9850 2800
@@
 	9850 2350 9850 2800
 $Comp
-L power:GND #PWR?
+L power:GND #PWR0126
 U 1 1 5FE49B06
 P 10300 3150
-F 0 "#PWR?" H 10300 2900 50  0001 C CNN
+F 0 "#PWR0126" H 10300 2900 50  0001 C CNN
 F 1 "GND" H 10305 2977 50  0000 C CNN
 F 2 "" H 10300 3150 50  0001 C CNN
@@
 P 8700 2550
 F 0 "C26" H 8792 2596 50  0000 L CNN
-F 1 "10nF" H 8792 2505 50  0000 L CNN
+F 1 "10nF 16V" H 8792 2505 50  0000 L CNN
 F 2 "Capacitor_SMD:C_0603_1608Metric" H 8700 2550 50  0001 C CNN
 F 3 "~" H 8700 2550 50  0001 C CNN
@@
 Connection ~ 2150 3050
 $Comp
-L power:GND #PWR?
+L power:GND #PWR0127
 U 1 1 5FE824E0
 P 3300 3350
-F 0 "#PWR?" H 3300 3100 50  0001 C CNN
+F 0 "#PWR0127" H 3300 3100 50  0001 C CNN
 F 1 "GND" H 3305 3177 50  0000 C CNN
 F 2 "" H 3300 3350 50  0001 C CNN
@@
 	3300 3250 3300 3350
 $Comp
-L power:GND #PWR?
+L power:GND #PWR0128
 U 1 1 5FE85C43
 P 4800 3750
-F 0 "#PWR?" H 4800 3500 50  0001 C CNN
+F 0 "#PWR0128" H 4800 3500 50  0001 C CNN
 F 1 "GND" H 4805 3577 50  0000 C CNN
 F 2 "" H 4800 3750 50  0001 C CNN
@@
 	1    0    0    -1
 $EndComp
+Wire Wire Line
+	7150 2800 7150 2700
+Wire Wire Line
+	7150 2700 7650 2700
+Connection ~ 7150 2700
+Wire Wire Line
+	7650 2900 7650 3100
+Wire Wire Line
+	7650 3100 7150 3100
+Wire Wire Line
+	7150 3100 7150 3000
+NoConn ~ 1450 3250
 $EndSCHEMATC

Commit message: improved +5V supply visibility
Other:
- moved on the sheet: C21, C22, C23, C27, D1, D2, J6, L1, R22, R23, R24, U8

Commit message: fixed -3V supply
Parts:
- L3: value L -> 4.7uH 4R7
Connections:
- net +5V: now also C5.2, R37.2, U9.5 (IN)
- net at C3.2, R37.1, U9.4 (EN): now also U9.3 (VIN); no longer U9.5 (IN)
Other:
- moved on the sheet: C10, C2, C21, C22, C23, C25, C26, C27, C3, C4, C5, C6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

Commit message: changed -3V3 power supply
Parts:
- removed C10: 4.7nF, symbol Device:C_Small
- removed C2: 0.22uF, symbol Device:C_Small
- removed C3: 0.1uF, symbol Device:C_Small
- removed C4: 10pF, symbol Device:C_Small
- removed C5: 10uF, symbol Device:C_Small
- removed C6, C7, C8, C9: 4.7uF, symbol Device:C_Small
- removed D7: SL03-GS08, symbol Device:D_Schottky
- removed L3: 4.7uH 4R7, symbol Device:L
- removed R36: 150k, symbol Device:R
- removed R37: 10R, symbol Device:R
- removed R38: 410k, symbol Device:R
- removed R39: 100k, symbol Device:R
- removed U9: TPS63700DRCT, DRC10_2P4X1P65, symbol TPS63700:TPS63700DRCT
- added C? (x2): 22uF, symbol Device:C_Small
- added C?: 2.2uF, symbol Device:C_Small
- added C?: 1000pF, symbol Device:C_Small
- added D?: MBR0520, Diode_SMD:D_SOD-123, symbol Diode:MBR0520
- added L? (x2): 22uH, symbol Device:L
- added R?: 16.83k 1%, Resistor_SMD:R_0603_1608Metric, symbol Device:R_Small
- added R?: 10k 1%, Resistor_SMD:R_0603_1608Metric, symbol Device:R_Small
- added U?: LM2611xMF, Package_TO_SOT_SMD:SOT-23-5, symbol Regulator_Switching:LM2611xMF
- L1: value SRR0604-100ML -> 4.7uH 1.2A
- R24: value 10k -> 10k 1%
- R27: value 10.2k 1% -> 10k 1%
Connections:
- net +12V: now also C?.2, L?.2, U?.4 (~SHDN), U?.5 (VIN)
- net -3V3: now also C?.2, C?.2, L?.1, R?.1
- net GND: now also C?.1, C?.1, D?.1 (K), R?.2, U?.2 (GND)
- new net: C?.1, L?.1, U?.1 (SW)
- new net: C?.1, R?.1, R?.2, U?.3 (NFB)
- new net: C?.2, D?.2 (A), L?.2

Commit message: annotated sch
Parts:
- gave numbers to parts that had none: 10
Changed lines of the file:
@@
 $EndComp
 $Comp
-L Regulator_Switching:LM2611xMF U?
+L Regulator_Switching:LM2611xMF U9
 U 1 1 5FFD5FE5
 P 5400 4900
-F 0 "U?" H 5400 5267 50  0000 C CNN
+F 0 "U9" H 5400 5267 50  0000 C CNN
 F 1 "LM2611xMF" H 5400 5176 50  0000 C CNN
 F 2 "Package_TO_SOT_SMD:SOT-23-5" H 5450 4650 50  0001 L CNN
@@
 $EndComp
 $Comp
-L power:+12V #PWR?
+L power:+12V #PWR010
 U 1 1 5FFE5730
 P 4200 4250
-F 0 "#PWR?" H 4200 4100 50  0001 C CNN
+F 0 "#PWR010" H 4200 4100 50  0001 C CNN
 F 1 "+12V" H 4215 4423 50  0000 C CNN
 F 2 "" H 4200 4250 50  0001 C CNN
@@
 	5000 4800 4850 4800
 $Comp
-L Device:C_Small C?
+L Device:C_Small C3
 U 1 1 5FFEA55E
 P 4200 4350
-F 0 "C?" H 4108 4304 50  0000 R CNN
+F 0 "C3" H 4108 4304 50  0000 R CNN
 F 1 "22uF" H 4108 4395 50  0000 R CNN
 F 2 "" H 4200 4350 50  0001 C CNN
@@
 Connection ~ 4200 4250
 $Comp
-L power:GND #PWR?
+L power:GND #PWR028
 U 1 1 5FFEB2C2
 P 4200 4450
-F 0 "#PWR?" H 4200 4200 50  0001 C CNN
+F 0 "#PWR028" H 4200 4200 50  0001 C CNN
 F 1 "GND" H 4205 4277 50  0000 C CNN
 F 2 "" H 4200 4450 50  0001 C CNN
@@
 $EndComp
 $Comp
-L power:GND #PWR?
+L power:GND #PWR029
 U 1 1 5FFEB990
 P 5400 5200
-F 0 "#PWR?" H 5400 4950 50  0001 C CNN
+F 0 "#PWR029" H 5400 4950 50  0001 C CNN
 F 1 "GND" H 5405 5027 50  0000 C CNN
 F 2 "" H 5400 5200 50  0001 C CNN
@@
 	4850 4250 4200 4250
 $Comp
-L Device:L L?
+L Device:L L3
 U 1 1 5FFF027B
 P 5400 4250
-F 0 "L?" V 5222 4250 50  0000 C CNN
+F 0 "L3" V 5222 4250 50  0000 C CNN
 F 1 "22uH" V 5313 4250 50  0000 C CNN
 F 2 "" H 5400 4250 50  0001 C CNN
@@
 	6000 4800 5800 4800
 $Comp
-L Device:C_Small C?
+L Device:C_Small C2
 U 1 1 6000090C
 P 6250 4250
-F 0 "C?" V 6500 4300 50  0000 R CNN
+F 0 "C2" V 6500 4300 50  0000 R CNN
 F 1 "2.2uF" V 6400 4300 50  0000 R CNN
 F 2 "" H 6250 4250 50  0001 C CNN
@@
 $EndComp
 $Comp
-L Diode:MBR0520 D?
+L Diode:MBR0520 D7
 U 1 1 600087BE
 P 7300 4700
-F 0 "D?" V 7346 4620 50  0000 R CNN
+F 0 "D7" V 7346 4620 50  0000 R CNN
 F 1 "MBR0520" V 7255 4620 50  0000 R CNN
 F 2 "Diode_SMD:D_SOD-123" H 7300 4525 50  0001 C CNN
@@
 $EndComp
 $Comp
-L Device:L L?
+L Device:L L4
 U 1 1 6000BFB1
 P 7550 4250
-F 0 "L?" V 7372 4250 50  0000 C CNN
+F 0 "L4" V 7372 4250 50  0000 C CNN
 F 1 "22uH" V 7463 4250 50  0000 C CNN
 F 2 "" H 7550 4250 50  0001 C CNN
@@
 $EndComp
 $Comp
-L Device:C_Small C?
+L Device:C_Small C5
 U 1 1 60016AA7
 P 7900 4700
-F 0 "C?" H 7808 4654 50  0000 R CNN
+F 0 "C5" H 7808 4654 50  0000 R CNN
 F 1 "22uF" H 7808 4745 50  0000 R CNN
 F 2 "" H 7900 4700 50  0001 C CNN
@@
 	7700 4250 7900 4250
 $Comp
-L Device:R_Small R?
+L Device:R_Small R16
 U 1 1 60028691
 P 6750 4700
-F 0 "R?" H 6809 4746 50  0000 L CNN
+F 0 "R16" H 6809 4746 50  0000 L CNN
 F 1 "16.83k 1%" H 6809 4655 50  0000 L CNN
 F 2 "Resistor_SMD:R_0603_1608Metric" H 6750 4700 50  0001 C CNN
@@
 $EndComp
 $Comp
-L Device:R_Small R?
+L Device:R_Small R17
 U 1 1 6003A1FB
 P 6750 5150
-F 0 "R?" H 6809 5196 50  0000 L CNN
+F 0 "R17" H 6809 5196 50  0000 L CNN
 F 1 "10k 1%" H 6809 5105 50  0000 L CNN
 F 2 "Resistor_SMD:R_0603_1608Metric" H 6750 5150 50  0001 C CNN
@@
 	7900 4250 7900 4450
 $Comp
-L power:GND #PWR?
+L power:GND #PWR030
 U 1 1 6004A3F0
 P 7600 5350
-F 0 "#PWR?" H 7600 5100 50  0001 C CNN
+F 0 "#PWR030" H 7600 5100 50  0001 C CNN
 F 1 "GND" H 7605 5177 50  0000 C CNN
 F 2 "" H 7600 5350 50  0001 C CNN
@@
 Connection ~ 7300 5350
 $Comp
-L Device:C_Small C?
+L Device:C_Small C4
 U 1 1 60056F7A
 P 6250 4700
-F 0 "C?" H 6158 4654 50  0000 R CNN
+F 0 "C4" H 6158 4654 50  0000 R CNN
 F 1 "1000pF" H 6158 4745 50  0000 R CNN
 F 2 "" H 6250 4700 50  0001 C CNN
@@
 Connection ~ 7900 4450
 $Comp
-L power:-3V3 #PWR?
+L power:-3V3 #PWR019
 U 1 1 60080D7B
 P 7900 4250
-F 0 "#PWR?" H 7900 4350 50  0001 C CNN
+F 0 "#PWR019" H 7900 4350 50  0001 C CNN
 F 1 "-3V3" H 7915 4423 50  0000 C CNN
 F 2 "" H 7900 4250 50  0001 C CNN
