File: Hardware/Power.sch (KiCad schematic (older format))
At the start: 32 parts, among them J6 Barrel_Jack_MountingPin, U10 LM2734Y, U8 LM2734Y, U9 LM2611xMF

Commit message: ERC check on the schematics
Changed lines of the file:
@@
 L power:+9V #PWR021
 U 1 1 5D1829E8
-P 10200 2050
-F 0 "#PWR021" H 10200 1900 50  0001 C CNN
-F 1 "+9V" H 10215 2223 50  0000 C CNN
-F 2 "" H 10200 2050 50  0001 C CNN
-F 3 "" H 10200 2050 50  0001 C CNN
-	1    10200 2050
+P 10200 1900
+F 0 "#PWR021" H 10200 1750 50  0001 C CNN
+F 1 "+9V" H 10215 2073 50  0000 C CNN
+F 2 "" H 10200 1900 50  0001 C CNN
+F 3 "" H 10200 1900 50  0001 C CNN
+	1    10200 1900
 	1    0    0    -1
 $EndComp
@@
 $EndComp
 Wire Wire Line
-	10200 2050 10200 2100
+	10200 1900 10200 2100
 Wire Wire Line
 	10200 2100 9750 2100

Commit message: added footprints to components
Parts:
- C2, C4: footprint (none) -> Capacitor_SMD:C_0603_1608Metric
- C3, C5: footprint (none) -> Capacitor_SMD:C_0805_2012Metric
- J6: value Barrel_Jack_MountingPin -> 694106301002; footprint (none) -> Connector_BarrelJack:BarrelJack_Wuerth_6941xx301002
- L3, L4: footprint (none) -> Inductor_SMD:L_Taiyo-Yuden_NR-60xx_HandSoldering
Changed lines of the file:
@@
 P 1350 2100
 F 0 "J6" H 1405 2417 50  0000 C CNN
-F 1 "Barrel_Jack_MountingPin" H 1405 2326 50  0000 C CNN
-F 2 "" H 1400 2060 50  0001 C CNN
+F 1 "694106301002" H 1405 2326 50  0000 C CNN
+F 2 "Connector_BarrelJack:BarrelJack_Wuerth_6941xx301002" H 1400 2060 50  0001 C CNN
 F 3 "~" H 1400 2060 50  0001 C CNN
 	1    1350 2100
@@
 F 0 "C3" H 4108 4304 50  0000 R CNN
 F 1 "22uF" H 4108 4395 50  0000 R CNN
-F 2 "" H 4200 4350 50  0001 C CNN
+F 2 "Capacitor_SMD:C_0805_2012Metric" H 4200 4350 50  0001 C CNN
 F 3 "~" H 4200 4350 50  0001 C CNN
 	1    4200 4350
@@
 F 0 "L3" V 5222 4250 50  0000 C CNN
 F 1 "22uH" V 5313 4250 50  0000 C CNN
-F 2 "" H 5400 4250 50  0001 C CNN
+F 2 "Inductor_SMD:L_Taiyo-Yuden_NR-60xx_HandSoldering" H 5400 4250 50  0001 C CNN
 F 3 "~" H 5400 4250 50  0001 C CNN
 	1    5400 4250
@@
 F 0 "C2" V 6500 4300 50  0000 R CNN
 F 1 "2.2uF" V 6400 4300 50  0000 R CNN
-F 2 "" H 6250 4250 50  0001 C CNN
+F 2 "Capacitor_SMD:C_0603_1608Metric" H 6250 4250 50  0001 C CNN
 F 3 "~" H 6250 4250 50  0001 C CNN
 	1    6250 4250
@@
 F 0 "L4" V 7372 4250 50  0000 C CNN
 F 1 "22uH" V 7463 4250 50  0000 C CNN
-F 2 "" H 7550 4250 50  0001 C CNN
+F 2 "Inductor_SMD:L_Taiyo-Yuden_NR-60xx_HandSoldering" H 7550 4250 50  0001 C CNN
 F 3 "~" H 7550 4250 50  0001 C CNN
 	1    7550 4250
@@
 F 0 "C5" H 7808 4654 50  0000 R CNN
 F 1 "22uF" H 7808 4745 50  0000 R CNN
-F 2 "" H 7900 4700 50  0001 C CNN
+F 2 "Capacitor_SMD:C_0805_2012Metric" H 7900 4700 50  0001 C CNN
 F 3 "~" H 7900 4700 50  0001 C CNN
 	1    7900 4700
@@
 F 0 "C4" H 6158 4654 50  0000 R CNN
 F 1 "1000pF" H 6158 4745 50  0000 R CNN
-F 2 "" H 6250 4700 50  0001 C CNN
+F 2 "Capacitor_SMD:C_0603_1608Metric" H 6250 4700 50  0001 C CNN
 F 3 "~" H 6250 4700 50  0001 C CNN
 	1    6250 4700

Commit message: swapped current sensing opamps for better routing
Parts:
- C21, C27: footprint Capacitor_SMD:C_0603_1608Metric -> Capacitor_SMD:C_0805_2012Metric
- C23: footprint Capacitor_SMD:C_0603_1608Metric -> Capacitor_SMD:C_1206_3216Metric
- C3, C5: footprint Capacitor_SMD:C_0805_2012Metric -> Capacitor_SMD:C_1206_3216Metric
- D2, D4: value SS1P3L -> CRS08; footprint Diode_SMD:D_SMA -> Diode_SMD:D_SOD-123F
- L1: footprint Inductor_SMD:L_6.3x6.3_H3 -> Inductor_SMD:L_Taiyo-Yuden_NR-40xx; MPN (none) -> NR4018T4R7M
- L2: value 22uH 1.4 A -> 22uH 1.4A; footprint Inductor_SMD:L_7.3x7.3_H3.5 -> Inductor_SMD:L_Taiyo-Yuden_NR-50xx; MPN SLF7045T-220M1R3-1PF -> NRS5040T220MMGKV
- L3, L4: value 22uH -> 22uH 1.4A; footprint Inductor_SMD:L_Taiyo-Yuden_NR-60xx_HandSoldering -> Inductor_SMD:L_Taiyo-Yuden_NR-50xx; MPN (none) -> NRS5040T220MMGKV
Changed lines of the file:
@@
 F 0 "C21" H 2142 2146 50  0000 L CNN
 F 1 "10uF" H 2142 2055 50  0000 L CNN
-F 2 "Capacitor_SMD:C_0603_1608Metric" H 2050 2100 50  0001 C CNN
+F 2 "Capacitor_SMD:C_0805_2012Metric" H 2050 2100 50  0001 C CNN
 F 3 "~" H 2050 2100 50  0001 C CNN
 	1    2050 2100
@@
 F 0 "L1" V 4322 2100 50  0000 C CNN
 F 1 "4.7uH 1.2A" V 4413 2100 50  0000 C CNN
-F 2 "Inductor_SMD:L_6.3x6.3_H3" H 4500 2100 50  0001 C CNN
+F 2 "Inductor_SMD:L_Taiyo-Yuden_NR-40xx" H 4500 2100 50  0001 C CNN
 F 3 "~" H 4500 2100 50  0001 C CNN
+F 4 "NR4018T4R7M" V 4500 2100 50  0001 C CNN "MPN"
 	1    4500 2100
 	0    1    1    0
@@
 P 4000 2300
 F 0 "D2" V 3954 2379 50  0000 L CNN
-F 1 "SS1P3L" V 4045 2379 50  0000 L CNN
-F 2 "Diode_SMD:D_SMA" H 4000 2300 50  0001 C CNN
+F 1 "CRS08" V 4045 2379 50  0000 L CNN
+F 2 "Diode_SMD:D_SOD-123F" H 4000 2300 50  0001 C CNN
 F 3 "~" H 4000 2300 50  0001 C CNN
 	1    4000 2300
@@
 	-1   0    0    1
 $EndComp
-$Comp
-L Device:L L2
-U 1 1 5D152A1F
-P 8950 2100
-F 0 "L2" V 8850 2100 50  0000 C CNN
-F 1 "22uH 1.4 A" V 9050 2200 50  0000 C CNN
-F 2 "Inductor_SMD:L_7.3x7.3_H3.5" H 8950 2100 50  0001 C CNN
-F 3 "~" H 8950 2100 50  0001 C CNN
-F 4 "SLF7045T-220M1R3-1PF" V 8950 2100 50  0001 C CNN "MPN"
-	1    8950 2100
-	0    1    1    0
-$EndComp
 Wire Wire Line
 	6700 1950 6700 2000
@@
 F 0 "C27" H 10292 2246 50  0000 L CNN
 F 1 "22uF 16V" H 10292 2155 50  0000 L CNN
-F 2 "Capacitor_SMD:C_0603_1608Metric" H 10200 2200 50  0001 C CNN
+F 2 "Capacitor_SMD:C_0805_2012Metric" H 10200 2200 50  0001 C CNN
 F 3 "~" H 10200 2200 50  0001 C CNN
 	1    10200 2200
@@
 P 8600 2300
 F 0 "D4" V 8554 2379 50  0000 L CNN
-F 1 "SS1P3L" V 8645 2379 50  0000 L CNN
-F 2 "Diode_SMD:D_SMA" H 8600 2300 50  0001 C CNN
+F 1 "CRS08" V 8645 2379 50  0000 L CNN
+F 2 "Diode_SMD:D_SOD-123F" H 8600 2300 50  0001 C CNN
 F 3 "~" H 8600 2300 50  0001 C CNN
 	1    8600 2300
@@
 F 0 "C23" H 5692 2296 50  0000 L CNN
 F 1 "22uF" H 5692 2205 50  0000 L CNN
-F 2 "Capacitor_SMD:C_0603_1608Metric" H 5600 2250 50  0001 C CNN
+F 2 "Capacitor_SMD:C_1206_3216Metric" H 5600 2250 50  0001 C CNN
 F 3 "~" H 5600 2250 50  0001 C CNN
 	1    5600 2250
@@
 F 0 "C3" H 4108 4304 50  0000 R CNN
 F 1 "22uF" H 4108 4395 50  0000 R CNN
-F 2 "Capacitor_SMD:C_0805_2012Metric" H 4200 4350 50  0001 C CNN
+F 2 "Capacitor_SMD:C_1206_3216Metric" H 4200 4350 50  0001 C CNN
 F 3 "~" H 4200 4350 50  0001 C CNN
 	1    4200 4350
@@
 P 5400 4250
 F 0 "L3" V 5222 4250 50  0000 C CNN
-F 1 "22uH" V 5313 4250 50  0000 C CNN
-F 2 "Inductor_SMD:L_Taiyo-Yuden_NR-60xx_HandSoldering" H 5400 4250 50  0001 C CNN
+F 1 "22uH 1.4A" V 5313 4250 50  0000 C CNN
+F 2 "Inductor_SMD:L_Taiyo-Yuden_NR-50xx" H 5400 4250 50  0001 C CNN
 F 3 "~" H 5400 4250 50  0001 C CNN
+F 4 "NRS5040T220MMGKV" V 5400 4250 50  0001 C CNN "MPN"
 	1    5400 4250
 	0    1    1    0
@@
 $EndComp
 $Comp
-L Device:L L4
-U 1 1 6000BFB1
-P 7550 4250
-F 0 "L4" V 7372 4250 50  0000 C CNN
-F 1 "22uH" V 7463 4250 50  0000 C CNN
-F 2 "Inductor_SMD:L_Taiyo-Yuden_NR-60xx_HandSoldering" H 7550 4250 50  0001 C CNN
-F 3 "~" H 7550 4250 50  0001 C CNN
-	1    7550 4250
-	0    1    1    0
-$EndComp
-$Comp
 L Device:C_Small C5
 U 1 1 60016AA7
@@
 F 0 "C5" H 7808 4654 50  0000 R CNN
 F 1 "22uF" H 7808 4745 50  0000 R CNN
-F 2 "Capacitor_SMD:C_0805_2012Metric" H 7900 4700 50  0001 C CNN
+F 2 "Capacitor_SMD:C_1206_3216Metric" H 7900 4700 50  0001 C CNN
 F 3 "~" H 7900 4700 50  0001 C CNN
 	1    7900 4700
@@
 $EndComp
 Connection ~ 4850 4250
+$Comp
+L Device:L L4
+U 1 1 6010A5B9
+P 7550 4250
+F 0 "L4" V 7372 4250 50  0000 C CNN
+F 1 "22uH 1.4A" V 7463 4250 50  0000 C CNN
+F 2 "Inductor_SMD:L_Taiyo-Yuden_NR-50xx" H 7550 4250 50  0001 C CNN
+F 3 "~" H 7550 4250 50  0001 C CNN
+F 4 "NRS5040T220MMGKV" V 7550 4250 50  0001 C CNN "MPN"
+	1    7550 4250
+	0    1    1    0
+$EndComp
+$Comp
+L Device:L L2
+U 1 1 6010D800
+P 8950 2100
+F 0 "L2" V 8900 2150 50  0000 C CNN
+F 1 "22uH 1.4A" V 9050 2200 50  0000 C CNN
+F 2 "Inductor_SMD:L_Taiyo-Yuden_NR-50xx" H 8950 2100 50  0001 C CNN
+F 3 "~" H 8950 2100 50  0001 C CNN
+F 4 "NRS5040T220MMGKV" V 8950 2100 50  0001 C CNN "MPN"
+	1    8950 2100
+	0    1    1    0
+$EndComp
 $EndSCHEMATC
