File: Hardware/STM32.sch (KiCad schematic (older format))
At the start: 14 parts

Commit message: added dissipation Mosfet, cleaned up Main sheet
Connections:
- net ADC-SHUNT: now reaches U?.17 (PA3)
- net OCStatus: now reaches U?.20 (PA4)
- net OCControl: now reaches U?.21 (PA5)
Changed lines of the file:
@@
 $Descr A4 11693 8268
 encoding utf-8
-Sheet 2 4
+Sheet 2 5
 Title ""
 Date ""
@@
 Wire Wire Line
 	6400 3650 7350 3650
+Text HLabel 7350 2550 2    50   Input ~ 0
+ADC-SHUNT
+Wire Wire Line
+	7350 2550 6400 2550
+Text HLabel 7350 2650 2    50   Input ~ 0
+OCStatus
+Text HLabel 7350 2750 2    50   Input ~ 0
+OCControl
+Wire Wire Line
+	6400 2650 7350 2650
+Wire Wire Line
+	6400 2750 7350 2750
 $EndSCHEMATC

Commit message: cleaned up power supplies
Changed lines of the file:
@@
 Wire Wire Line
 	6400 2750 7350 2750
+Text GLabel 5150 1600 1    50   Input ~ 0
++3.3V
+Wire Wire Line
+	5150 1600 5150 1750
+Text GLabel 4150 5650 0    50   Input ~ 0
+GND
 $EndSCHEMATC

Commit message: cleanup main sheet+added temperature measurement
Connections:
- net TempSense: now reaches U?.22 (PA6)
Changed lines of the file:
@@
 Text GLabel 4150 5650 0    50   Input ~ 0
 GND
+Text HLabel 7350 2850 2    50   Input ~ 0
+TempSense
+Wire Wire Line
+	7350 2850 6400 2850
 $EndSCHEMATC

Commit message: error check on schematic done
Parts:
- gave numbers to parts that had none: 14
Changed lines of the file:
@@
 $EndDescr
 $Comp
-L power:+3.3V #PWR?
+L power:+3.3V #PWR08
 U 1 1 5D0488F4
 P 5500 1750
-F 0 "#PWR?" H 5500 1600 50  0001 C CNN
+F 0 "#PWR08" H 5500 1600 50  0001 C CNN
 F 1 "+3.3V" H 5515 1923 50  0000 C CNN
 F 2 "" H 5500 1750 50  0001 C CNN
@@
 $EndComp
 $Comp
-L MCU_ST_STM32F4:STM32F446RETx U?
+L MCU_ST_STM32F4:STM32F446RETx U3
 U 1 1 5D048902
 P 5700 3750
-F 0 "U?" H 5700 1861 50  0000 C CNN
+F 0 "U3" H 5700 1861 50  0000 C CNN
 F 1 "STM32F446RETx" H 5700 1770 50  0000 C CNN
 F 2 "Package_QFP:LQFP-64_10x10mm_P0.5mm" H 5100 2050 50  0001 R CNN
@@
 DAC-D7
 $Comp
-L power:GND #PWR?
+L power:GND #PWR010
 U 1 1 5D048931
 P 6300 5650
-F 0 "#PWR?" H 6300 5400 50  0001 C CNN
+F 0 "#PWR010" H 6300 5400 50  0001 C CNN
 F 1 "GND" H 6305 5477 50  0000 C CNN
 F 2 "" H 6300 5650 50  0001 C CNN
@@
 Connection ~ 5500 1750
 $Comp
-L power:+3.3VADC #PWR?
+L power:+3.3VADC #PWR09
 U 1 1 5D048952
 P 6150 1750
-F 0 "#PWR?" H 6300 1700 50  0001 C CNN
+F 0 "#PWR09" H 6300 1700 50  0001 C CNN
 F 1 "+3.3VADC" H 6170 1893 50  0000 C CNN
 F 2 "" H 6150 1750 50  0001 C CNN
@@
 	6000 1750 6150 1750
 $Comp
-L Device:C C?
+L Device:C C14
 U 1 1 5D04895A
 P 5150 1900
-F 0 "C?" V 4898 1900 50  0000 C CNN
+F 0 "C14" V 4898 1900 50  0000 C CNN
 F 1 "100nF" V 4989 1900 50  0000 C CNN
 F 2 "" H 5188 1750 50  0001 C CNN
@@
 $EndComp
 $Comp
-L Device:C C?
+L Device:C C13
 U 1 1 5D048960
 P 4750 1900
-F 0 "C?" V 4498 1900 50  0000 C CNN
+F 0 "C13" V 4498 1900 50  0000 C CNN
 F 1 "100nF" V 4589 1900 50  0000 C CNN
 F 2 "" H 4788 1750 50  0001 C CNN
@@
 $EndComp
 $Comp
-L Device:C C?
+L Device:C C11
 U 1 1 5D048966
 P 4350 1900
-F 0 "C?" V 4098 1900 50  0000 C CNN
+F 0 "C11" V 4098 1900 50  0000 C CNN
 F 1 "100nF" V 4189 1900 50  0000 C CNN
 F 2 "" H 4388 1750 50  0001 C CNN
@@
 $EndComp
 $Comp
-L Device:C C?
+L Device:C C8
 U 1 1 5D04896C
 P 3950 1900
-F 0 "C?" V 3698 1900 50  0000 C CNN
+F 0 "C8" V 3698 1900 50  0000 C CNN
 F 1 "100nF" V 3789 1900 50  0000 C CNN
 F 2 "" H 3988 1750 50  0001 C CNN
@@
 	4750 1750 5150 1750
 $Comp
-L Device:C C?
+L Device:C C15
 U 1 1 5D048974
 P 6300 1900
-F 0 "C?" V 6048 1900 50  0000 C CNN
+F 0 "C15" V 6048 1900 50  0000 C CNN
 F 1 "10nF" V 6139 1900 50  0000 C CNN
 F 2 "" H 6338 1750 50  0001 C CNN
@@
 $EndComp
 $Comp
-L Device:C C?
+L Device:C C16
 U 1 1 5D04897A
 P 6700 1900
-F 0 "C?" V 6448 1900 50  0000 C CNN
+F 0 "C16" V 6448 1900 50  0000 C CNN
 F 1 "1uF" V 6539 1900 50  0000 C CNN
 F 2 "" H 6738 1750 50  0001 C CNN
@@
 	6300 2050 6550 2050
 $Comp
-L power:GND #PWR?
+L power:GND #PWR011
 U 1 1 5D048985
 P 6550 2050
-F 0 "#PWR?" H 6550 1800 50  0001 C CNN
+F 0 "#PWR011" H 6550 1800 50  0001 C CNN
 F 1 "GND" H 6555 1877 50  0000 C CNN
 F 2 "" H 6550 2050 50  0001 C CNN
@@
 	6550 2050 6700 2050
 $Comp
-L Device:Crystal_Small Y?
+L Device:Crystal_Small Y1
 U 1 1 5D04898D
 P 4750 3400
-F 0 "Y?" H 4750 3625 50  0000 C CNN
+F 0 "Y1" H 4750 3625 50  0000 C CNN
 F 1 "ABM7-8.000MHZ-D2Y-T" H 4750 3534 50  0000 C CNN
 F 2 "" H 4750 3400 50  0001 C CNN
@@
 	4750 2050 5150 2050
 $Comp
-L power:GND #PWR?
+L power:GND #PWR07
 U 1 1 5D04899E
 P 4550 2050
-F 0 "#PWR?" H 4550 1800 50  0001 C CNN
+F 0 "#PWR07" H 4550 1800 50  0001 C CNN
 F 1 "GND" H 4555 1877 50  0000 C CNN
 F 2 "" H 4550 2050 50  0001 C CNN
@@
 	4550 2050 4750 2050
 $Comp
-L Device:C C?
+L Device:C C9
 U 1 1 5D0489A6
 P 4300 3300
-F 0 "C?" V 4048 3300 50  0000 C CNN
+F 0 "C9" V 4048 3300 50  0000 C CNN
 F 1 "20pF" V 4139 3300 50  0000 C CNN
 F 2 "" H 4338 3150 50  0001 C CNN
@@
 $EndComp
 $Comp
-L Device:C C?
+L Device:C C10
 U 1 1 5D0489AC
 P 4300 3500
-F 0 "C?" V 4048 3500 50  0000 C CNN
+F 0 "C10" V 4048 3500 50  0000 C CNN
 F 1 "20pF" V 4139 3500 50  0000 C CNN
 F 2 "" H 4338 3350 50  0001 C CNN
@@
 Connection ~ 4150 3500
 $Comp
-L Device:C C?
+L Device:C C12
 U 1 1 5D0489BE
 P 4500 2650
-F 0 "C?" V 4248 2650 50  0000 C CNN
+F 0 "C12" V 4248 2650 50  0000 C CNN
 F 1 "4.7uF" V 4339 2650 50  0000 C CNN
 F 2 "" H 4538 2500 50  0001 C CNN
@@
 	4650 2650 5000 2650
 $Comp
-L Device:R R?
+L Device:R R9
 U 1 1 5D0489C8
 P 4800 2450
-F 0 "R?" H 4870 2496 50  0000 L CNN
+F 0 "R9" H 4870 2496 50  0000 L CNN
 F 1 "1k" H 4870 2405 50  0000 L CNN
 F 2 "" V 4730 2450 50  0001 C CNN
@@
 Connection ~ 4150 2650
 $Comp
-L Device:R R?
+L Device:R R8
 U 1 1 5D0489D2
 P 3750 2100
-F 0 "R?" H 3820 2146 50  0000 L CNN
+F 0 "R8" H 3820 2146 50  0000 L CNN
 F 1 "4.7k" H 3820 2055 50  0000 L CNN
 F 2 "" V 3680 2100 50  0001 C CNN
@@
 Connection ~ 3950 1750
 $Comp
-L Switch:SW_Push SW?
+L Switch:SW_Push SW1
 U 1 1 5D0489DB
 P 3750 2450
-F 0 "SW?" V 3704 2598 50  0000 L CNN
+F 0 "SW1" V 3704 2598 50  0000 L CNN
 F 1 "SW_Push" V 3795 2598 50  0000 L CNN
 F 2 "" H 3750 2650 50  0001 C CNN
