File: Hardware/Laser-Driver-v2.sch (KiCad schematic (older format))
At the start: 36 parts

Commit message: power supplies added
Parts:
- R?: value 7k -> 12k
Other:
- note added: "Internal Gain: 2.5"
- note added: "Second stage amplifier:\nGain 13"
- moved on the sheet: R?
Changed lines of the file:
@@
 EESchema Schematic File Version 4
-EELAYER 29 0
+EELAYER 26 0
 EELAYER END
 $Descr A4 11693 8268
 encoding utf-8
-Sheet 1 3
+Sheet 1 4
 Title ""
 Date ""
@@
 L Device:R R?
 U 1 1 5CDE8E37
-P 5500 1950
-F 0 "R?" H 5570 1996 50  0000 L CNN
-F 1 "1k" H 5570 1905 50  0000 L CNN
-F 2 "" V 5430 1950 50  0001 C CNN
-F 3 "~" H 5500 1950 50  0001 C CNN
-	1    5500 1950
+P 5450 1950
+F 0 "R?" H 5520 1996 50  0000 L CNN
+F 1 "1k" H 5520 1905 50  0000 L CNN
+F 2 "" V 5380 1950 50  0001 C CNN
+F 3 "~" H 5450 1950 50  0001 C CNN
+	1    5450 1950
 	-1   0    0    1
 $EndComp
@@
 L Device:R R?
 U 1 1 5CDE7B2D
-P 5500 1650
-F 0 "R?" H 5570 1696 50  0000 L CNN
-F 1 "7k" H 5570 1605 50  0000 L CNN
-F 2 "" V 5430 1650 50  0001 C CNN
-F 3 "~" H 5500 1650 50  0001 C CNN
-	1    5500 1650
-	1    0    0    -1
-$EndComp
-Wire Wire Line
-	5500 1500 5850 1500
+P 5450 1650
+F 0 "R?" H 5520 1696 50  0000 L CNN
+F 1 "12k" H 5520 1605 50  0000 L CNN
+F 2 "" V 5380 1650 50  0001 C CNN
+F 3 "~" H 5450 1650 50  0001 C CNN
+	1    5450 1650
+	1    0    0    -1
+$EndComp
 $Comp
 L Device:R R?
@@
 L power:GND #PWR?
 U 1 1 5CDED2D0
-P 5750 2150
-F 0 "#PWR?" H 5750 1900 50  0001 C CNN
-F 1 "GND" H 5755 1977 50  0000 C CNN
-F 2 "" H 5750 2150 50  0001 C CNN
-F 3 "" H 5750 2150 50  0001 C CNN
-	1    5750 2150
+P 5750 2300
+F 0 "#PWR?" H 5750 2050 50  0001 C CNN
+F 1 "GND" H 5755 2127 50  0000 C CNN
+F 2 "" H 5750 2300 50  0001 C CNN
+F 3 "" H 5750 2300 50  0001 C CNN
+	1    5750 2300
 	1    0    0    -1
 $EndComp
@@
 Connection ~ 6850 1700
 Wire Wire Line
-	5500 2100 5750 2100
+	5450 2100 5750 2100
 Connection ~ 5750 2100
 Wire Wire Line
-	5750 2100 5750 2150
-Wire Wire Line
-	5500 1800 5650 1800
+	5750 2100 5750 2300
 Wire Wire Line
 	5650 1800 5650 2000
-Connection ~ 5500 1800
 Wire Wire Line
 	5200 3700 5200 1500
 Wire Wire Line
-	5200 1500 5500 1500
-Connection ~ 5500 1500
+	5200 1500 5450 1500
 Wire Wire Line
 	5750 4600 6050 4600
@@
 Wire Wire Line
 	9500 4700 9700 4700
+$Sheet
+S 8550 1150 1150 1000
+U 5D12441E
+F0 "Power" 50
+F1 "Power.sch" 50
+$EndSheet
+Text Notes 2250 1600 0    50   ~ 0
+Internal Gain: 2.5
+Text Notes 5850 2200 0    50   ~ 0
+Second stage amplifier:\nGain 13
+Connection ~ 5450 1500
+Wire Wire Line
+	5450 1500 5850 1500
+Connection ~ 5450 1800
+Wire Wire Line
+	5450 1800 5650 1800
 $EndSCHEMATC

Commit message: added dissipation Mosfet, cleaned up Main sheet
Parts:
- removed C? (x4): 100nF, symbol Device:C
- removed D?: TLLR4400, symbol Device:LED
- removed Q?: BSS138, Package_TO_SOT_SMD:SOT-23, symbol Transistor_FET:BSS138
- removed R? (x3): 56K, symbol Device:R
- removed R?: 50K, symbol Device:R
- removed R?: 10K, symbol Device:R
- removed R?: 166R, symbol Device:R
- removed R?: 1,55K, symbol Device:R
- removed RV?: 10K, symbol Device:R_POT_TRIM
- removed SW?: SW_Push, symbol Switch:SW_Push
- removed U?: TC75S57F, symbol OS-LD:TC75S57F
- removed U?: TC4452, Package_SO:SOIC-8_3.9x4.9mm_P1.27mm, symbol OS-LD:TC4452
- removed U?: LM285D-1.2, Package_SO:SOIC-8_3.9x4.9mm_P1.27mm, symbol Reference_Voltage:LM285D-1.2
- removed U? (x2): 74LVC2G02, symbol 74xGxx:74LVC2G02
- removed U?: 74LVC1G08, symbol 74xGxx:74LVC1G08
- removed U?: 74AHCT1G04, symbol 74xGxx:74AHCT1G04
- added Q?: IRFP4568PbF, Package_TO_SOT_THT:TO-247-3_Vertical, symbol OS-LD:IRFP4568PbF
- added R?: R_Shunt, symbol Device:R_Shunt
Connections:
- net Vi is gone; now on an unnamed net: R?.1
- net +5V: now also C?.1; no longer C?.2
- net GND: now also C?.1, C?.1, C?.2, R?.1; no longer C?.1, C?.2, C?.2
- net Output Stage/MOSFET-OUT: now also Q?.1 (G)
- net at U?.5 (RS+): now also R?.3
- net at U?.6 (RS-): now also R?.2
- net STM32 Schematic/ADC-SHUNT: now reaches R?.1, U?.1 (OUT)
- net at R?.1: now also U?.8 (OUT); no longer U?.3 (+IN)
- net at Q?.1 (S), Q?.2 (S), Q?.3 (S): now also R?.4
- net Overcurrent Protection/OCMosfet: now reaches Q?.4 (G)
- net at Q?.5 (D): now also Q?.3 (S)
- new net: C?.2, C?.2, U?.2 (Vee)
- new net: R?.2, U?.3 (+IN)
- new net Overcurrent Protection/OCSense: R?.2
Other:
- note removed: "Overcurrent Protection Circuit"
- note removed: "RS-Latch"
- note removed: "Reset Logic Circuit"
- note removed: "SET=1, IF Vref>Vi"
- moved on the sheet: C?, Q?, R?, U?

Commit message: cleaned up power supplies
Changed lines of the file:
@@
 	1750 3000 2250 3000
 $Sheet
-S 8550 3350 600  500
+S 8550 3350 1050 650
 U 5D12441E
 F0 "Power" 50
 F1 "Power.sch" 50
 F2 "+12V" I L 8550 3450 50
-F3 "GND" I R 9150 3450 50
-F4 "+5V" I L 8550 3650 50
-F5 "+3.3V" I L 8550 3750 50
-F6 "+9V" I L 8550 3550 50
+F3 "GND" I R 9600 3450 50
+F4 "+5V" I L 8550 3750 50
+F5 "+3.3V" I L 8550 3900 50
+F6 "+9V" I L 8550 3600 50
 $EndSheet
 Text Notes 4100 7050 0    50   ~ 0
@@
 Wire Wire Line
 	1950 3350 1750 3350
-Text GLabel 8450 3450 0    50   Input ~ 0
-+12V
-Text GLabel 8450 3550 0    50   Input ~ 0
-+9V
-Text GLabel 8450 3650 0    50   Input ~ 0
-+5V
-Text GLabel 8450 3750 0    50   Input ~ 0
-+3.3V
-Text GLabel 9250 3450 2    50   Input ~ 0
-GND
-Wire Wire Line
-	8450 3450 8550 3450
-Wire Wire Line
-	8450 3550 8550 3550
-Wire Wire Line
-	8450 3650 8550 3650
-Wire Wire Line
-	8450 3750 8550 3750
 Connection ~ 5500 3000
 Wire Wire Line
 	5500 3000 5500 2900
-Wire Wire Line
-	9150 3450 9250 3450
 $Comp
 L power:+5V #PWR?

Commit message: cleanup main sheet+added temperature measurement
Parts:
- added C?: 100nF, symbol Device:C
- added J? (x4): 74650074R, symbol Connector:Screw_Terminal_01x01
- added J?: Screw_Terminal_01x02, symbol Connector:Screw_Terminal_01x02
- added R?: 10k, symbol Device:R
- added TH?: NTCALUG03A103G, symbol Device:Thermistor
Connections:
- net GND: now also C?.1, J?.1 (Pin_1), J?.1 (Pin_1), J?.1 (Pin_1)
- net at Q?.2 (D): now also J?.1 (Pin_1), J?.1 (Pin_1)
- new net: TH?.1, TH?.2
- new net +3V3: R?.2
- new net STM32 Schematic/OCStatus: C?.2, J?.2 (Pin_2), R?.1
Other:
- note added: "OFFBOARD!!!"
- moved on the sheet: C?, Q?, R?, U?

Commit message: error check on schematic done
Parts:
- gave numbers to parts that had none: 24
Connections:
- net STM32 Schematic/OCStatus renamed STM32 Schematic/TempSense
Other:
- moved on the sheet: R6
Changed lines of the file:
@@
 $EndDescr
 $Comp
-L OS-LD:MAX9643 U?
+L OS-LD:MAX9643 U1
 U 1 1 5CDC6E2E
 P 4150 6450
-F 0 "U?" H 4150 6127 50  0000 C CNN
+F 0 "U1" H 4150 6127 50  0000 C CNN
 F 1 "MAX9643" H 4150 6036 50  0000 C CNN
 F 2 "" H 4150 6150 50  0001 C CNN
@@
 $EndComp
 $Comp
-L Device:C C?
+L Device:C C3
 U 1 1 5CDC76E9
 P 3250 6550
-F 0 "C?" H 3365 6596 50  0000 L CNN
+F 0 "C3" H 3365 6596 50  0000 L CNN
 F 1 "1uF" H 3365 6505 50  0000 L CNN
 F 2 "" H 3288 6400 50  0001 C CNN
@@
 	3750 6300 3750 6050
 $Comp
-L power:+5V #PWR?
+L power:+5V #PWR04
 U 1 1 5CDE0555
 P 4950 5900
-F 0 "#PWR?" H 4950 5750 50  0001 C CNN
+F 0 "#PWR04" H 4950 5750 50  0001 C CNN
 F 1 "+5V" H 4965 6073 50  0000 C CNN
 F 2 "" H 4950 5900 50  0001 C CNN
@@
 $EndComp
 $Comp
-L Device:C C?
+L Device:C C7
 U 1 1 5CDEE828
 P 5200 3650
-F 0 "C?" V 4948 3650 50  0000 C CNN
+F 0 "C7" V 4948 3650 50  0000 C CNN
 F 1 "100nF" V 5039 3650 50  0000 C CNN
 F 2 "" H 5238 3500 50  0001 C CNN
@@
 $EndComp
 $Comp
-L Device:R R?
+L Device:R R4
 U 1 1 5CDFB610
 P 4300 4000
-F 0 "R?" V 4093 4000 50  0000 C CNN
+F 0 "R4" V 4093 4000 50  0000 C CNN
 F 1 "1k" V 4184 4000 50  0000 C CNN
 F 2 "" V 4230 4000 50  0001 C CNN
@@
 $EndComp
 $Comp
-L Device:R R?
+L Device:R R6
 U 1 1 5CDFBA7F
-P 4750 4000
-F 0 "R?" V 4543 4000 50  0000 C CNN
-F 1 "1k" V 4634 4000 50  0000 C CNN
-F 2 "" V 4680 4000 50  0001 C CNN
-F 3 "~" H 4750 4000 50  0001 C CNN
-	1    4750 4000
+P 4800 4000
+F 0 "R6" V 4593 4000 50  0000 C CNN
+F 1 "1k" V 4684 4000 50  0000 C CNN
+F 2 "" V 4730 4000 50  0001 C CNN
+F 3 "~" H 4800 4000 50  0001 C CNN
+	1    4800 4000
 	0    1    1    0
 $EndComp
 $Comp
-L Device:C C?
+L Device:C C5
 U 1 1 5CDFBC7C
 P 4550 4150
-F 0 "C?" H 4665 4196 50  0000 L CNN
+F 0 "C5" H 4665 4196 50  0000 L CNN
 F 1 "10pF" H 4665 4105 50  0000 L CNN
 F 2 "" H 4588 4000 50  0001 C CNN
@@
 	4450 4000 4550 4000
 Wire Wire Line
-	4550 4000 4600 4000
-$Comp
-L power:GND #PWR?
+	4550 4000 4650 4000
+$Comp
+L power:GND #PWR03
 U 1 1 5CE00065
 P 4550 4350
-F 0 "#PWR?" H 4550 4100 50  0001 C CNN
+F 0 "#PWR03" H 4550 4100 50  0001 C CNN
 F 1 "GND" H 4555 4177 50  0000 C CNN
 F 2 "" H 4550 4350 50  0001 C CNN
@@
 	4550 4300 4550 4350
 $Comp
-L Device:R R?
+L Device:R R5
 U 1 1 5CE06C26
 P 4400 5500
-F 0 "R?" H 4330 5454 50  0000 R CNN
+F 0 "R5" H 4330 5454 50  0000 R CNN
 F 1 "1k" H 4330 5545 50  0000 R CNN
 F 2 "" V 4330 5500 50  0001 C CNN
@@
 	4200 2950 4200 2750
 $Comp
-L Device:R R?
+L Device:R R3
 U 1 1 5CDE8E37
 P 3650 3200
-F 0 "R?" H 3720 3246 50  0000 L CNN
+F 0 "R3" H 3720 3246 50  0000 L CNN
 F 1 "1k" H 3720 3155 50  0000 L CNN
 F 2 "" V 3580 3200 50  0001 C CNN
@@
 $EndComp
 $Comp
-L Device:R R?
+L Device:R R2
 U 1 1 5CDE7B2D
 P 3650 2900
-F 0 "R?" H 3720 2946 50  0000 L CNN
+F 0 "R2" H 3720 2946 50  0000 L CNN
 F 1 "12k" H 3720 2855 50  0000 L CNN
 F 2 "" V 3580 2900 50  0001 C CNN
@@
 	3650 6400 3750 6400
 $Comp
-L Device:C C?
+L Device:C C2
 U 1 1 5CDC7B44
 P 2850 6950
-F 0 "C?" H 2965 6996 50  0000 L CNN
+F 0 "C2" H 2965 6996 50  0000 L CNN
 F 1 "100nF" H 2965 6905 50  0000 L CNN
 F 2 "" H 2888 6800 50  0001 C CNN
@@
 $EndComp
 $Comp
-L Device:C C?
+L Device:C C4
 U 1 1 5CDC7F91
 P 3300 6950
-F 0 "C?" H 3415 6996 50  0000 L CNN
+F 0 "C4" H 3415 6996 50  0000 L CNN
 F 1 "1uF" H 3415 6905 50  0000 L CNN
 F 2 "" H 3338 6800 50  0001 C CNN
@@
 	3650 6300 3650 6400
 $Comp
-L power:GND #PWR?
+L power:GND #PWR06
 U 1 1 5CDC96ED
 P 6150 7300
-F 0 "#PWR?" H 6150 7050 50  0001 C CNN
+F 0 "#PWR06" H 6150 7050 50  0001 C CNN
 F 1 "GND" H 6155 7127 50  0000 C CNN
 F 2 "" H 6150 7300 50  0001 C CNN
@@
 $EndComp
 $Comp
-L OS-LD:PSMN0R7-25YLD Q?
+L OS-LD:PSMN0R7-25YLD Q2
 U 1 1 5CE09D45
 P 6050 5900
-F 0 "Q?" H 6256 5946 50  0000 L CNN
+F 0 "Q2" H 6256 5946 50  0000 L CNN
 F 1 "PSMN0R7-25YLD" H 6256 5855 50  0000 L CNN
 F 2 "Package_TO_SOT_SMD:LFPAK56" H 6200 5900 50  0001 C CNN
@@
 $EndComp
 $Comp
-L OS-LD:TVL3541 U?
+L OS-LD:TVL3541 U2
 U 1 1 5D151151
 P 4500 3050
-F 0 "U?" H 4500 3375 50  0000 C CNN
+F 0 "U2" H 4500 3375 50  0000 C CNN
 F 1 "TLV3541" H 4500 3284 50  0000 C CNN
 F 2 "" H 4500 3050 50  0001 C CNN
@@
 F16 "DAC-CLOCK" I R 1600 2950 50
 F17 "ADC-SHUNT" I R 1600 3100 50
-F18 "OCSense" I R 1600 3200 50
+F18 "OCStatus" I R 1600 3200 50
 F19 "OCControl" I R 1600 3300 50
-F20 "OCStatus" I R 1600 3400 50
+F20 "TempSense" I R 1600 3400 50
 $EndSheet
 $Sheet
@@
 Second stage amplifier:\nGain 13
 $Comp
-L OS-LD:IRFP4568PbF Q?
+L OS-LD:IRFP4568PbF Q1
 U 1 1 5D20B94F
 P 6050 1500
-F 0 "Q?" H 6256 1546 50  0000 L CNN
+F 0 "Q1" H 6256 1546 50  0000 L CNN
 F 1 "IRFP4568PbF" H 6256 1455 50  0000 L CNN
 F 2 "Package_TO_SOT_THT:TO-247-3_Vertical" H 6200 1500 50  0001 C CNN
@@
 $EndSheet
 $Comp
-L Device:R_Shunt R?
+L Device:R_Shunt R7
 U 1 1 5D24ABAC
 P 6150 6600
-F 0 "R?" H 6063 6554 50  0000 R CNN
+F 0 "R7" H 6063 6554 50  0000 R CNN
 F 1 "R_Shunt" H 6063 6645 50  0000 R CNN
 F 2 "" V 6080 6600 50  0001 C CNN
@@
 	4550 5500 4650 5500
 $Comp
-L Device:C C?
+L Device:C C6
 U 1 1 5CDC899C
 P 4950 6950
-F 0 "C?" H 5065 6996 50  0000 L CNN
+F 0 "C6" H 5065 6996 50  0000 L CNN
 F 1 "100nF" H 5065 6905 50  0000 L CNN
 F 2 "" H 4988 6800 50  0001 C CNN
@@
 	4050 3150 4050 4000
 Wire Wire Line
-	5000 4000 4900 4000
+	5000 4000 4950 4000
 Wire Wire Line
 	5000 4000 5000 5500
@@
 	5200 2950 5200 2850
 $Comp
-L power:+5V #PWR?
+L power:+5V #PWR05
 U 1 1 5CDED736
 P 5200 2850
-F 0 "#PWR?" H 5200 2700 50  0001 C CNN
+F 0 "#PWR05" H 5200 2700 50  0001 C CNN
 F 1 "+5V" H 5215 3023 50  0000 C CNN
 F 2 "" H 5200 2850 50  0001 C CNN
@@
 Connection ~ 3650 3050
 $Comp
-L Connector:Screw_Terminal_01x01 J?
+L Connector:Screw_Terminal_01x01 J5
 U 1 1 5D38D38E
 P 6350 7200
-F 0 "J?" H 6430 7242 50  0000 L CNN
+F 0 "J5" H 6430 7242 50  0000 L CNN
 F 1 " 74650074R" H 6430 7151 50  0000 L CNN
 F 2 "" H 6350 7200 50  0001 C CNN
@@
 	6150 7200 6150 7300
 $Comp
-L Connector:Screw_Terminal_01x01 J?
+L Connector:Screw_Terminal_01x01 J4
 U 1 1 5D38D663
 P 6350 7050
-F 0 "J?" H 6430 7092 50  0000 L CNN
+F 0 "J4" H 6430 7092 50  0000 L CNN
 F 1 " 74650074R" H 6430 7001 50  0000 L CNN
 F 2 "" H 6350 7050 50  0001 C CNN
@@
 	6150 7050 6150 7200
 $Comp
-L Connector:Screw_Terminal_01x01 J?
+L Connector:Screw_Terminal_01x01 J3
 U 1 1 5D38D69B
 P 6350 1100
-F 0 "J?" H 6430 1142 50  0000 L CNN
+F 0 "J3" H 6430 1142 50  0000 L CNN
 F 1 " 74650074R" H 6430 1051 50  0000 L CNN
 F 2 "" H 6350 1100 50  0001 C CNN
@@
 $EndComp
 $Comp
-L Connector:Screw_Terminal_01x01 J?
+L Connector:Screw_Terminal_01x01 J2
 U 1 1 5D38D8B8
 P 6350 950
-F 0 "J?" H 6430 992 50  0000 L CNN
+F 0 "J2" H 6430 992 50  0000 L CNN
 F 1 " 74650074R" H 6430 901 50  0000 L CNN
 F 2 "" H 6350 950 50  0001 C CNN
@@
 	5850 1500 6000 1500
 $Comp
-L Device:Thermistor TH?
+L Device:Thermistor TH1
 U 1 1 5D39C944
 P 2100 5700
-F 0 "TH?" H 2205 5746 50  0000 L CNN
+F 0 "TH1" H 2205 5746 50  0000 L CNN
 F 1 "NTCALUG03A103G" H 2205 5655 50  0000 L CNN
 F 2 "" H 2100 5700 50  0001 C CNN
@@
 	2800 5600 3000 5600
 $Comp
-L Device:R R?
+L Device:R R1
 U 1 1 5D3A5AFA
 P 1250 5050
-F 0 "R?" H 1180 5004 50  0000 R CNN
+F 0 "R1" H 1180 5004 50  0000 R CNN
 F 1 "10k" H 1180 5095 50  0000 R CNN
 F 2 "" V 1180 5050 50  0001 C CNN
@@
 $EndComp
 $Comp
-L power:GND #PWR?
+L power:GND #PWR02
 U 1 1 5D3A5BD3
 P 1250 6050
-F 0 "#PWR?" H 1250 5800 50  0001 C CNN
+F 0 "#PWR02" H 1250 5800 50  0001 C CNN
 F 1 "GND" H 1255 5877 50  0000 C CNN
 F 2 "" H 1250 6050 50  0001 C CNN
@@
 $EndComp
 $Comp
-L Connector:Screw_Terminal_01x02 J?
+L Connector:Screw_Terminal_01x02 J1
 U 1 1 5D3A8C70
 P 1600 5600
-F 0 "J?" H 1519 5275 50  0000 C CNN
+F 0 "J1" H 1519 5275 50  0000 C CNN
 F 1 "Screw_Terminal_01x02" H 1519 5366 50  0000 C CNN
 F 2 "" H 1600 5600 50  0001 C CNN
@@
 +3.3V
 $Comp
-L power:+3.3V #PWR?
+L power:+3.3V #PWR01
 U 1 1 5D3C851F
 P 1250 4550
-F 0 "#PWR?" H 1250 4400 50  0001 C CNN
+F 0 "#PWR01" H 1250 4400 50  0001 C CNN
 F 1 "+3.3V" H 1265 4723 50  0000 C CNN
 F 2 "" H 1250 4550 50  0001 C CNN
@@
 	1600 5500 2100 5500
 $Comp
-L Device:C C?
+L Device:C C1
 U 1 1 5D3ECE3F
 P 900 5650
-F 0 "C?" H 1015 5696 50  0000 L CNN
+F 0 "C1" H 1015 5696 50  0000 L CNN
 F 1 "100nF" H 1015 5605 50  0000 L CNN
 F 2 "" H 938 5500 50  0001 C CNN
@@
 Wire Wire Line
 	900  5950 1250 5950
+Wire Wire Line
+	1250 5950 1250 6050
 Connection ~ 1250 5950
-Wire Wire Line
-	1250 5950 1250 6050
 Text Notes 2200 5850 0    50   ~ 0
 OFFBOARD!!!

Commit message: footprint for M4 screw terminal added to schematic
Parts:
- J2, J3, J4, J5: footprint (none) -> OS-LD:WP-THRBU
Changed lines of the file:
@@
 Wire Wire Line
 	3800 3050 3800 3250
-Text Notes 5550 500  0    50   ~ 0
+Text Notes 3900 2400 0    50   ~ 0
 Alternative for TLV3541: THS4271
 $Sheet
@@
 F 0 "J5" H 6430 7242 50  0000 L CNN
 F 1 " 74650074R" H 6430 7151 50  0000 L CNN
-F 2 "" H 6350 7200 50  0001 C CNN
+F 2 "OS-LD:WP-THRBU" H 6350 7200 50  0001 C CNN
 F 3 "~" H 6350 7200 50  0001 C CNN
 	1    6350 7200
@@
 F 0 "J4" H 6430 7092 50  0000 L CNN
 F 1 " 74650074R" H 6430 7001 50  0000 L CNN
-F 2 "" H 6350 7050 50  0001 C CNN
+F 2 "OS-LD:WP-THRBU" H 6350 7050 50  0001 C CNN
 F 3 "~" H 6350 7050 50  0001 C CNN
 	1    6350 7050
@@
 F 0 "J3" H 6430 1142 50  0000 L CNN
 F 1 " 74650074R" H 6430 1051 50  0000 L CNN
-F 2 "" H 6350 1100 50  0001 C CNN
+F 2 "OS-LD:WP-THRBU" H 6350 1100 50  0001 C CNN
 F 3 "~" H 6350 1100 50  0001 C CNN
 	1    6350 1100
@@
 F 0 "J2" H 6430 992 50  0000 L CNN
 F 1 " 74650074R" H 6430 901 50  0000 L CNN
-F 2 "" H 6350 950 50  0001 C CNN
+F 2 "OS-LD:WP-THRBU" H 6350 950 50  0001 C CNN
 F 3 "~" H 6350 950 50  0001 C CNN
 	1    6350 950
