File: Hardware/Overcurrent.sch (KiCad schematic (older format))
At the start: 20 parts, among them Q3 BSS138, U11 LM285D-1.2, U12 74LVC2G04, U13 74LVC1G08, U14 TC75S57F, U15 74LVC2G02, U16 TC4452

Commit message: ERC check on the schematics
Parts:
- gave numbers to parts that had none: 1
Changed lines of the file:
@@
 P 2500 6000
 AR Path="/60057FD1" Ref="SW?"  Part="1"
-AR Path="/5D20CDF9/60057FD1" Ref="SW?"  Part="1"
-F 0 "SW?" H 2500 6285 50  0000 C CNN
+AR Path="/5D20CDF9/60057FD1" Ref="SW1"  Part="1"
+F 0 "SW1" H 2500 6285 50  0000 C CNN
 F 1 "SW_Push" H 2500 6194 50  0000 C CNN
 F 2 "" H 2500 6200 50  0001 C CNN
@@
 P 2900 6500
 AR Path="/6005AB7C" Ref="#PWR?"  Part="1"
-AR Path="/5D20CDF9/6005AB7C" Ref="#PWR?"  Part="1"
-F 0 "#PWR?" H 2900 6250 50  0001 C CNN
+AR Path="/5D20CDF9/6005AB7C" Ref="#PWR048"  Part="1"
+F 0 "#PWR048" H 2900 6250 50  0001 C CNN
 F 1 "GND" H 2905 6327 50  0000 C CNN
 F 2 "" H 2900 6500 50  0001 C CNN
@@
 P 2150 5950
 AR Path="/6005CF78" Ref="#PWR?"  Part="1"
-AR Path="/5D20CDF9/6005CF78" Ref="#PWR?"  Part="1"
-F 0 "#PWR?" H 2150 5800 50  0001 C CNN
+AR Path="/5D20CDF9/6005CF78" Ref="#PWR047"  Part="1"
+F 0 "#PWR047" H 2150 5800 50  0001 C CNN
 F 1 "+5V" H 2165 6123 50  0000 C CNN
 F 2 "" H 2150 5950 50  0001 C CNN
@@
 P 3200 5250
 AR Path="/60062CB2" Ref="#PWR?"  Part="1"
-AR Path="/5D20CDF9/60062CB2" Ref="#PWR?"  Part="1"
-F 0 "#PWR?" H 3200 5000 50  0001 C CNN
+AR Path="/5D20CDF9/60062CB2" Ref="#PWR045"  Part="1"
+F 0 "#PWR045" H 3200 5000 50  0001 C CNN
 F 1 "GND" H 3205 5077 50  0000 C CNN
 F 2 "" H 3200 5250 50  0001 C CNN
@@
 P 4400 4500
 AR Path="/600641F4" Ref="#PWR?"  Part="1"
-AR Path="/5D20CDF9/600641F4" Ref="#PWR?"  Part="1"
-F 0 "#PWR?" H 4400 4250 50  0001 C CNN
+AR Path="/5D20CDF9/600641F4" Ref="#PWR042"  Part="1"
+F 0 "#PWR042" H 4400 4250 50  0001 C CNN
 F 1 "GND" H 4405 4327 50  0000 C CNN
 F 2 "" H 4400 4500 50  0001 C CNN
@@
 P 3200 4950
 AR Path="/6006D7F3" Ref="#PWR?"  Part="1"
-AR Path="/5D20CDF9/6006D7F3" Ref="#PWR?"  Part="1"
-F 0 "#PWR?" H 3200 4800 50  0001 C CNN
+AR Path="/5D20CDF9/6006D7F3" Ref="#PWR043"  Part="1"
+F 0 "#PWR043" H 3200 4800 50  0001 C CNN
 F 1 "+5V" H 3215 5123 50  0000 C CNN
 F 2 "" H 3200 4950 50  0001 C CNN
@@
 P 4400 4250
 AR Path="/6007056A" Ref="#PWR?"  Part="1"
-AR Path="/5D20CDF9/6007056A" Ref="#PWR?"  Part="1"
-F 0 "#PWR?" H 4400 4100 50  0001 C CNN
+AR Path="/5D20CDF9/6007056A" Ref="#PWR041"  Part="1"
+F 0 "#PWR041" H 4400 4100 50  0001 C CNN
 F 1 "+5V" H 4415 4423 50  0000 C CNN
 F 2 "" H 4400 4250 50  0001 C CNN
@@
 P 4400 5100
 AR Path="/60095275" Ref="#PWR?"  Part="1"
-AR Path="/5D20CDF9/60095275" Ref="#PWR?"  Part="1"
-F 0 "#PWR?" H 4400 4950 50  0001 C CNN
+AR Path="/5D20CDF9/60095275" Ref="#PWR044"  Part="1"
+F 0 "#PWR044" H 4400 4950 50  0001 C CNN
 F 1 "+5V" H 4415 5273 50  0000 C CNN
 F 2 "" H 4400 5100 50  0001 C CNN
@@
 P 4400 5300
 AR Path="/60095997" Ref="#PWR?"  Part="1"
-AR Path="/5D20CDF9/60095997" Ref="#PWR?"  Part="1"
-F 0 "#PWR?" H 4400 5050 50  0001 C CNN
+AR Path="/5D20CDF9/60095997" Ref="#PWR046"  Part="1"
+F 0 "#PWR046" H 4400 5050 50  0001 C CNN
 F 1 "GND" H 4405 5127 50  0000 C CNN
 F 2 "" H 4400 5300 50  0001 C CNN

Commit message: added footprints to components
Parts:
- SW1: value SW_Push -> TL3305A; footprint (none) -> Button_Switch_SMD:SW_SPST_TL3305A
- U12: footprint (none) -> Package_TO_SOT_SMD:SOT-23-6_Handsoldering
- U13: value 74LVC1G08 -> SN74LVC1G08DBVR; footprint (none) -> Package_TO_SOT_SMD:SOT-23-5_HandSoldering
- U14: value TC75S57F -> TC75S57FU(TE85L,F); footprint (none) -> Package_TO_SOT_SMD:SOT-353_SC-70-5
- U15: footprint (none) -> Package_SO:SSOP-8_2.95x2.8mm_P0.65mm
Changed lines of the file:
@@
 AR Path="/5D20CDF9/5D223265" Ref="U14"  Part="1"
 F 0 "U14" H 4350 3165 50  0000 C CNN
-F 1 "TC75S57F" H 4350 3074 50  0000 C CNN
-F 2 "" V 3800 2350 50  0001 C CNN
+F 1 "TC75S57FU(TE85L,F)" H 4350 3074 50  0000 C CNN
+F 2 "Package_TO_SOT_SMD:SOT-353_SC-70-5" V 3800 2350 50  0001 C CNN
 F 3 "https://www.mouser.de/datasheet/2/408/TC75S57F_datasheet_en_20140301-760810.pdf" V 3800 2350 50  0001 C CNN
 	1    4350 2750
@@
 AR Path="/5D20CDF9/5D223297" Ref="U13"  Part="1"
 F 0 "U13" H 3100 5300 50  0000 C CNN
-F 1 "74LVC1G08" H 3175 5326 50  0001 C CNN
-F 2 "" H 3200 5150 50  0001 C CNN
+F 1 "SN74LVC1G08DBVR" H 3175 5326 50  0001 C CNN
+F 2 "Package_TO_SOT_SMD:SOT-23-5_HandSoldering" H 3200 5150 50  0001 C CNN
 F 3 "http://www.ti.com/lit/sg/scyt129e/scyt129e.pdf" H 3200 5150 50  0001 C CNN
 	1    3200 5150
@@
 F 0 "U15" H 4550 4550 50  0000 C CNN
 F 1 "74LVC2G02" H 4375 4576 50  0001 C CNN
-F 2 "" H 4400 4400 50  0001 C CNN
+F 2 "Package_SO:SSOP-8_2.95x2.8mm_P0.65mm" H 4400 4400 50  0001 C CNN
 F 3 "http://www.ti.com/lit/sg/scyt129e/scyt129e.pdf" H 4400 4400 50  0001 C CNN
 	2    4400 4400
@@
 F 0 "U15" H 4550 5350 50  0000 C CNN
 F 1 "74LVC2G02" H 4375 5376 50  0001 C CNN
-F 2 "" H 4400 5200 50  0001 C CNN
+F 2 "Package_SO:SSOP-8_2.95x2.8mm_P0.65mm" H 4400 5200 50  0001 C CNN
 F 3 "http://www.ti.com/lit/sg/scyt129e/scyt129e.pdf" H 4400 5200 50  0001 C CNN
 	1    4400 5200
@@
 F 0 "U12" H 5300 5000 50  0000 C CNN
 F 1 "74LVC2G04" H 5125 5026 50  0001 C CNN
-F 2 "" H 5150 4850 50  0001 C CNN
+F 2 "Package_TO_SOT_SMD:SOT-23-6_Handsoldering" H 5150 4850 50  0001 C CNN
 F 3 "http://www.ti.com/lit/sg/scyt129e/scyt129e.pdf" H 5150 4850 50  0001 C CNN
 	2    5150 4850
@@
 F 0 "U12" H 2350 5000 50  0000 C CNN
 F 1 "74LVC2G04" H 2625 5276 50  0001 C CNN
-F 2 "" H 2650 5100 50  0001 C CNN
+F 2 "Package_TO_SOT_SMD:SOT-23-6_Handsoldering" H 2650 5100 50  0001 C CNN
 F 3 "http://www.ti.com/lit/sg/scyt129e/scyt129e.pdf" H 2650 5100 50  0001 C CNN
 	1    2650 5100
@@
 AR Path="/5D20CDF9/60057FD1" Ref="SW1"  Part="1"
 F 0 "SW1" H 2500 6285 50  0000 C CNN
-F 1 "SW_Push" H 2500 6194 50  0000 C CNN
-F 2 "" H 2500 6200 50  0001 C CNN
+F 1 "TL3305A" H 2500 6194 50  0000 C CNN
+F 2 "Button_Switch_SMD:SW_SPST_TL3305A" H 2500 6200 50  0001 C CNN
 F 3 "~" H 2500 6200 50  0001 C CNN
 	1    2500 6000

Commit message: finished placement. started routing
Parts:
- added D8: RED, LED_SMD:LED_0603_1608Metric, symbol Device:LED
- added R36: 1k, Resistor_SMD:R_0603_1608Metric, symbol Device:R
- D6: value TLLR4400 -> GREEN; footprint LED_THT:LED_D3.0mm -> LED_SMD:LED_0603_1608Metric; MPN (none) -> LTST-C191KGKT
- R31: value 1,55K -> 1k
- RV1: footprint Potentiometer_THT:Potentiometer_ACP_CA9-V10_Vertical -> Potentiometer_SMD:Potentiometer_Bourns_3314G_Vertical; MPN (none) -> 3314G-1-103E
Connections:
- net GND: now also D8.1 (K)
- net at U12.3, U15.6, U15.7: now also R36.2
- new net: D8.2 (A), R36.1
Other:
- moved on the sheet: U12B
Changed lines of the file:
@@
 AR Path="/5D20CDF9/5D22333B" Ref="R31"  Part="1"
 F 0 "R31" H 6180 5104 50  0000 R CNN
-F 1 "1,55K" H 6180 5195 50  0000 R CNN
+F 1 "1k" H 6180 5195 50  0000 R CNN
 F 2 "Resistor_SMD:R_0603_1608Metric" V 6180 5150 50  0001 C CNN
 F 3 "~" H 6250 5150 50  0001 C CNN
@@
 F 0 "RV1" H 3031 2646 50  0000 R CNN
 F 1 "10K" H 3031 2555 50  0000 R CNN
-F 2 "Potentiometer_THT:Potentiometer_ACP_CA9-V10_Vertical" H 3100 2600 50  0001 C CNN
+F 2 "Potentiometer_SMD:Potentiometer_Bourns_3314G_Vertical" H 3100 2600 50  0001 C CNN
 F 3 "~" H 3100 2600 50  0001 C CNN
+F 4 "3314G-1-103E" H 3100 2600 50  0001 C CNN "MPN"
 	1    3100 2600
 	1    0    0    -1
@@
 AR Path="/5D20CDF9/5D223334" Ref="D6"  Part="1"
 F 0 "D6" H 6243 5766 50  0000 C CNN
-F 1 "TLLR4400" H 6243 5675 50  0000 C CNN
-F 2 "LED_THT:LED_D3.0mm" H 6250 5550 50  0001 C CNN
+F 1 "GREEN" H 6243 5675 50  0000 C CNN
+F 2 "LED_SMD:LED_0603_1608Metric" H 6250 5550 50  0001 C CNN
 F 3 "~" H 6250 5550 50  0001 C CNN
+F 4 "LTST-C191KGKT" H 6250 5550 50  0001 C CNN "MPN"
 	1    6250 5550
 	0    -1   -1   0
@@
 L 74xGxx:74LVC2G04 U12
 U 2 1 5FFE78B2
-P 5150 4850
-F 0 "U12" H 5300 5000 50  0000 C CNN
-F 1 "74LVC2G04" H 5125 5026 50  0001 C CNN
-F 2 "Package_TO_SOT_SMD:SOT-23-6_Handsoldering" H 5150 4850 50  0001 C CNN
-F 3 "http://www.ti.com/lit/sg/scyt129e/scyt129e.pdf" H 5150 4850 50  0001 C CNN
-	2    5150 4850
+P 5350 4850
+F 0 "U12" H 5500 5000 50  0000 C CNN
+F 1 "74LVC2G04" H 5325 5026 50  0001 C CNN
+F 2 "Package_TO_SOT_SMD:SOT-23-6_Handsoldering" H 5350 4850 50  0001 C CNN
+F 3 "http://www.ti.com/lit/sg/scyt129e/scyt129e.pdf" H 5350 4850 50  0001 C CNN
+	2    5350 4850
 	1    0    0    -1
 $EndComp
@@
 L power:GND #PWR?
 U 1 1 5FFF94B7
-P 5150 4950
+P 5350 4950
 AR Path="/5FFF94B7" Ref="#PWR?"  Part="1"
 AR Path="/5D20CDF9/5FFF94B7" Ref="#PWR040"  Part="1"
-F 0 "#PWR040" H 5150 4700 50  0001 C CNN
-F 1 "GND" H 5155 4777 50  0000 C CNN
-F 2 "" H 5150 4950 50  0001 C CNN
-F 3 "" H 5150 4950 50  0001 C CNN
-	1    5150 4950
+F 0 "#PWR040" H 5350 4700 50  0001 C CNN
+F 1 "GND" H 5355 4777 50  0000 C CNN
+F 2 "" H 5350 4950 50  0001 C CNN
+F 3 "" H 5350 4950 50  0001 C CNN
+	1    5350 4950
 	1    0    0    -1
 $EndComp
@@
 	3800 2900 3800 1350
 Wire Wire Line
-	5400 4850 6250 4850
+	5600 4850 6250 4850
 Connection ~ 6250 4850
 Wire Notes Line
@@
 Connection ~ 4700 4850
 Wire Wire Line
-	4700 4850 4850 4850
+	4700 4850 5000 4850
 Wire Wire Line
 	3850 4450 3850 4850
@@
 $EndComp
 Wire Wire Line
-	5150 4700 5150 4750
+	5350 4700 5350 4750
 $Comp
 L power:+5V #PWR?
 U 1 1 5FFF6DD8
-P 5150 4700
+P 5350 4700
 AR Path="/5FFF6DD8" Ref="#PWR?"  Part="1"
 AR Path="/5D20CDF9/5FFF6DD8" Ref="#PWR039"  Part="1"
-F 0 "#PWR039" H 5150 4550 50  0001 C CNN
-F 1 "+5V" H 5165 4873 50  0000 C CNN
-F 2 "" H 5150 4700 50  0001 C CNN
-F 3 "" H 5150 4700 50  0001 C CNN
-	1    5150 4700
-	1    0    0    -1
-$EndComp
+F 0 "#PWR039" H 5350 4550 50  0001 C CNN
+F 1 "+5V" H 5365 4873 50  0000 C CNN
+F 2 "" H 5350 4700 50  0001 C CNN
+F 3 "" H 5350 4700 50  0001 C CNN
+	1    5350 4700
+	1    0    0    -1
+$EndComp
+$Comp
+L Device:LED D?
+U 1 1 60196A7C
+P 5000 5550
+AR Path="/60196A7C" Ref="D?"  Part="1"
+AR Path="/5D20CDF9/60196A7C" Ref="D8"  Part="1"
+F 0 "D8" H 4993 5766 50  0000 C CNN
+F 1 "RED" H 4993 5675 50  0000 C CNN
+F 2 "LED_SMD:LED_0603_1608Metric" H 5000 5550 50  0001 C CNN
+F 3 "~" H 5000 5550 50  0001 C CNN
+F 4 "LTST-C190KRKT" H 5000 5550 50  0001 C CNN "MPN"
+	1    5000 5550
+	0    -1   -1   0
+$EndComp
+$Comp
+L power:GND #PWR?
+U 1 1 60197492
+P 5000 5700
+AR Path="/60197492" Ref="#PWR?"  Part="1"
+AR Path="/5D20CDF9/60197492" Ref="#PWR054"  Part="1"
+F 0 "#PWR054" H 5000 5450 50  0001 C CNN
+F 1 "GND" H 5005 5527 50  0000 C CNN
+F 2 "" H 5000 5700 50  0001 C CNN
+F 3 "" H 5000 5700 50  0001 C CNN
+	1    5000 5700
+	1    0    0    -1
+$EndComp
+$Comp
+L Device:R R?
+U 1 1 60197B9A
+P 5000 5150
+AR Path="/60197B9A" Ref="R?"  Part="1"
+AR Path="/5D20CDF9/60197B9A" Ref="R36"  Part="1"
+F 0 "R36" H 4930 5104 50  0000 R CNN
+F 1 "1k" H 4930 5195 50  0000 R CNN
+F 2 "Resistor_SMD:R_0603_1608Metric" V 4930 5150 50  0001 C CNN
+F 3 "~" H 5000 5150 50  0001 C CNN
+	1    5000 5150
+	-1   0    0    1
+$EndComp
+Wire Wire Line
+	5000 5000 5000 4850
+Connection ~ 5000 4850
+Wire Wire Line
+	5000 4850 5050 4850
+Wire Wire Line
+	5000 5300 5000 5400
 $EndSCHEMATC
