File: Hardware/Laser-Driver-v3.sch (KiCad schematic (older format))
At the start: 24 parts, among them J1 Screw_Terminal_01x02, J2 74650074R, J3 74650074R, J4 74650074R, J5 74650074R, Q1 IRFP4568PbF, Q2 PSMN0R7-25YLD, U1 MAX9643, U2 TLV3541

Commit message: STM32 replaced by Teensy
STM32 replaced by Teensy. OPA2354 added as amplifier frontend. Tina-Spice simulation file for amplifier frontend added.
Parts:
- removed C2, C6: 100nF, Capacitor_SMD:C_0603_1608Metric, symbol Device:C
- removed C3, C4: 1uF, Capacitor_SMD:C_0603_1608Metric, symbol Device:C
- removed R2: 12k, Resistor_SMD:R_0603_1608Metric, symbol Device:R
- removed R5: 1k, Resistor_SMD:R_0603_1608Metric, symbol Device:R
- removed U1: MAX9643, symbol OS-LD:MAX9643
- removed U2: TLV3541, Package_TO_SOT_SMD:SOT-23-5, symbol OS-LD:TVL3541
- added R? (x3): 100R, Resistor_SMD:R_0603_1608Metric, symbol Device:R
- added R? (x2): 10k, Resistor_SMD:R_0603_1608Metric, symbol Device:R
- added R?: 20k, Resistor_SMD:R_0603_1608Metric, symbol Device:R
- added U?: OPA2354, symbol OS-LD:OPA2354
Connections:
- net labels added: -3V3
- wire segments 122 -> 111
- no-connect marks 1 -> 0
Other:
- note removed: "Internal Gain: 2.5"
- moved on the sheet: C5, C7, Q2, R3, R4, R6, R7

Commit message: external ADC added
Parts:
- removed C5: 10pF, Capacitor_SMD:C_0603_1608Metric, symbol Device:C
- removed C7: 100nF, Capacitor_SMD:C_0603_1608Metric, symbol Device:C
- removed R3, R4, R6: 1k, Resistor_SMD:R_0603_1608Metric, symbol Device:R
Connections:
- net labels removed: +5V
- wire segments 111 -> 88
Other:
- note removed: "Second stage amplifier:\nGain 13"
Changed lines of the file:
@@
 $EndDescr
-$Comp
-L Device:C C7
-U 1 1 5CDEE828
-P 10100 1950
-F 0 "C7" V 9848 1950 50  0000 C CNN
-F 1 "100nF" V 9939 1950 50  0000 C CNN
-F 2 "Capacitor_SMD:C_0603_1608Metric" H 10138 1800 50  0001 C CNN
-F 3 "~" H 10100 1950 50  0001 C CNN
-	1    10100 1950
-	1    0    0    -1
-$EndComp
-$Comp
-L Device:R R4
-U 1 1 5CDFB610
-P 9200 2300
-F 0 "R4" V 8993 2300 50  0000 C CNN
-F 1 "1k" V 9084 2300 50  0000 C CNN
-F 2 "Resistor_SMD:R_0603_1608Metric" V 9130 2300 50  0001 C CNN
-F 3 "~" H 9200 2300 50  0001 C CNN
-	1    9200 2300
-	0    1    1    0
-$EndComp
-$Comp
-L Device:R R6
-U 1 1 5CDFBA7F
-P 9700 2300
-F 0 "R6" V 9493 2300 50  0000 C CNN
-F 1 "1k" V 9584 2300 50  0000 C CNN
-F 2 "Resistor_SMD:R_0603_1608Metric" V 9630 2300 50  0001 C CNN
-F 3 "~" H 9700 2300 50  0001 C CNN
-	1    9700 2300
-	0    1    1    0
-$EndComp
-$Comp
-L Device:C C5
-U 1 1 5CDFBC7C
-P 9450 2450
-F 0 "C5" H 9565 2496 50  0000 L CNN
-F 1 "10pF" H 9565 2405 50  0000 L CNN
-F 2 "Capacitor_SMD:C_0603_1608Metric" H 9488 2300 50  0001 C CNN
-F 3 "~" H 9450 2450 50  0001 C CNN
-	1    9450 2450
-	1    0    0    -1
-$EndComp
-Wire Wire Line
-	9350 2300 9450 2300
-Wire Wire Line
-	9450 2300 9550 2300
-$Comp
-L power:GND #PWR03
-U 1 1 5CE00065
-P 9450 2650
-F 0 "#PWR03" H 9450 2400 50  0001 C CNN
-F 1 "GND" H 9455 2477 50  0000 C CNN
-F 2 "" H 9450 2650 50  0001 C CNN
-F 3 "" H 9450 2650 50  0001 C CNN
-	1    9450 2650
-	1    0    0    -1
-$EndComp
-Wire Wire Line
-	9450 2600 9450 2650
-$Comp
-L Device:R R3
-U 1 1 5CDE8E37
-P 8550 1500
-F 0 "R3" H 8620 1546 50  0000 L CNN
-F 1 "1k" H 8620 1455 50  0000 L CNN
-F 2 "Resistor_SMD:R_0603_1608Metric" V 8480 1500 50  0001 C CNN
-F 3 "~" H 8550 1500 50  0001 C CNN
-	1    8550 1500
-	-1   0    0    1
-$EndComp
 $Comp
 L power:GND #PWR06
@@
 	1    0    0    -1
 $EndComp
-Wire Wire Line
-	9100 1350 8800 1350
-Wire Wire Line
-	8800 1350 8800 1650
-Wire Wire Line
-	9700 1450 9700 1550
-Wire Wire Line
-	9700 1550 8700 1550
-Wire Wire Line
-	9700 1250 10100 1250
-Wire Wire Line
-	8550 1650 8800 1650
-Connection ~ 8800 1650
-Wire Wire Line
-	8700 1350 8700 1550
 Text Notes 3900 2400 0    50   ~ 0
 Alternative for TLV3541: THS4271
@@
 S 600  1400 1000 2150
 U 5D037190
-F0 "STM32 Schematic" 50
+F0 "Teensy" 50
 F1 "STM32.sch" 50
 F2 "DAC-D0" I R 1600 1500 50
@@
 F6 "-3.3V" I R 9300 3800 50
 $EndSheet
-Text Notes 9100 1750 0    50   ~ 0
-Second stage amplifier:\nGain 13
 $Comp
 L OS-LD:IRFP4568PbF Q1
@@
 Connection ~ 6150 7300
 Wire Wire Line
-	8550 1350 8700 1350
-Wire Wire Line
-	9100 1450 8950 1450
-Wire Wire Line
-	8950 1450 8950 2300
-Wire Wire Line
-	9900 2300 9850 2300
-Wire Wire Line
-	9900 2300 9900 3800
-Wire Wire Line
-	8950 2300 9050 2300
-Wire Wire Line
-	8800 2650 9450 2650
-Wire Wire Line
-	8800 1650 8800 2650
-Connection ~ 9450 2650
-Wire Wire Line
-	9450 2650 10100 2650
-Wire Wire Line
-	10100 2650 10100 2100
-Wire Wire Line
-	10100 1800 10100 1250
-Wire Wire Line
 	2000 3700 2000 3100
 Wire Wire Line
@@
 Wire Wire Line
 	1800 3300 1600 3300
-Connection ~ 10100 1250
-Wire Wire Line
-	10100 1250 10100 1150
-$Comp
-L power:+5V #PWR05
-U 1 1 5CDED736
-P 10100 1150
-F 0 "#PWR05" H 10100 1000 50  0001 C CNN
-F 1 "+5V" H 10115 1323 50  0000 C CNN
-F 2 "" H 10100 1150 50  0001 C CNN
-F 3 "" H 10100 1150 50  0001 C CNN
-	1    10100 1150
-	1    0    0    -1
-$EndComp
-Connection ~ 9450 2300
-Text GLabel 10250 1250 2    50   Input ~ 0
-+5V
-Wire Wire Line
-	10250 1250 10100 1250
 Text GLabel 1950 7300 0    50   Input ~ 0
 GND

Commit message: fixed file name. used kicad default gitignore
Parts:
- gave numbers to parts that had none: 7
Changed lines of the file:
@@
 U 5D037190
 F0 "Teensy" 50
-F1 "STM32.sch" 50
+F1 "controller.sch" 50
 F2 "DAC-D0" I R 1600 1500 50
 F3 "DAC-D1" I R 1600 1600 50
@@
 	5850 3900 4800 3900
 $Comp
-L OS-LD:OPA2354 U?
+L OS-LD:OPA2354 U1
 U 1 1 5F275BCA
 P 4700 5550
-F 0 "U?" H 4950 5687 60  0000 C CNN
+F 0 "U1" H 4950 5687 60  0000 C CNN
 F 1 "OPA2354" H 4950 5581 60  0000 C CNN
 F 2 "" H 4750 5550 60  0001 C CNN
@@
 $EndComp
 $Comp
-L Device:R R?
+L Device:R R4
 U 1 1 5F232CF4
 P 5700 5250
-F 0 "R?" H 5630 5204 50  0000 R CNN
+F 0 "R4" H 5630 5204 50  0000 R CNN
 F 1 "100R" H 5630 5295 50  0000 R CNN
 F 2 "Resistor_SMD:R_0603_1608Metric" V 5630 5250 50  0001 C CNN
@@
 $EndComp
 $Comp
-L Device:R R?
+L Device:R R5
 U 1 1 5F2352F4
 P 5700 5450
-F 0 "R?" H 5630 5404 50  0000 R CNN
+F 0 "R5" H 5630 5404 50  0000 R CNN
 F 1 "100R" H 5630 5495 50  0000 R CNN
 F 2 "Resistor_SMD:R_0603_1608Metric" V 5630 5450 50  0001 C CNN
@@
 	5550 5400 5550 5450
 $Comp
-L Device:R R?
+L Device:R R6
 U 1 1 5F25607D
 P 5000 5550
-F 0 "R?" H 4930 5504 50  0000 R CNN
+F 0 "R6" H 4930 5504 50  0000 R CNN
 F 1 "100R" H 4930 5595 50  0000 R CNN
 F 2 "Resistor_SMD:R_0603_1608Metric" V 4930 5550 50  0001 C CNN
@@
 	3800 5300 4000 5300
 $Comp
-L power:-3V3 #PWR?
+L power:-3V3 #PWR0101
 U 1 1 5F7D57D9
 P 3750 5100
-F 0 "#PWR?" H 3750 5200 50  0001 C CNN
+F 0 "#PWR0101" H 3750 5200 50  0001 C CNN
 F 1 "-3V3" H 3765 5273 50  0000 C CNN
 F 2 "" H 3750 5100 50  0001 C CNN
@@
 	3750 5100 4000 5100
 $Comp
-L power:+3.3V #PWR?
+L power:+3.3V #PWR0102
 U 1 1 5F7DD72F
 P 4100 5650
-F 0 "#PWR?" H 4100 5500 50  0001 C CNN
+F 0 "#PWR0102" H 4100 5500 50  0001 C CNN
 F 1 "+3.3V" H 4115 5823 50  0000 C CNN
 F 2 "" H 4100 5650 50  0001 C CNN
@@
 	5000 5400 5550 5400
 $Comp
-L Device:R R?
+L Device:R R3
 U 1 1 5F800785
 P 5350 5000
-F 0 "R?" H 5280 4954 50  0000 R CNN
+F 0 "R3" H 5280 4954 50  0000 R CNN
 F 1 "20k" H 5280 5045 50  0000 R CNN
 F 2 "Resistor_SMD:R_0603_1608Metric" V 5280 5000 50  0001 C CNN
@@
 $EndComp
 $Comp
-L Device:R R?
+L Device:R R8
 U 1 1 5F8011C2
 P 5350 5650
-F 0 "R?" H 5280 5604 50  0000 R CNN
+F 0 "R8" H 5280 5604 50  0000 R CNN
 F 1 "10k" H 5280 5695 50  0000 R CNN
 F 2 "Resistor_SMD:R_0603_1608Metric" V 5280 5650 50  0001 C CNN
@@
 $EndComp
 $Comp
-L power:GND #PWR?
+L power:GND #PWR0103
 U 1 1 5F801827
 P 5350 5850
-F 0 "#PWR?" H 5350 5600 50  0001 C CNN
+F 0 "#PWR0103" H 5350 5600 50  0001 C CNN
 F 1 "GND" H 5355 5677 50  0000 C CNN
 F 2 "" H 5350 5850 50  0001 C CNN
@@
 	5350 5800 5350 5850
 $Comp
-L Device:R R?
+L Device:R R2
 U 1 1 5F6D354D
 P 4950 4200
-F 0 "R?" H 4880 4154 50  0000 R CNN
+F 0 "R2" H 4880 4154 50  0000 R CNN
 F 1 "10k" H 4880 4245 50  0000 R CNN
 F 2 "Resistor_SMD:R_0603_1608Metric" V 4880 4200 50  0001 C CNN

Commit message: removed labels from power connections. powr conn already global
Changed lines of the file:
@@
 Wire Wire Line
 	1250 5500 1250 5200
-Text GLabel 1500 4750 2    50   Input ~ 0
-+3.3V
 $Comp
 L power:+3.3V #PWR01
@@
 	1    0    0    -1
 $EndComp
-Wire Wire Line
-	1250 4900 1250 4750
-Wire Wire Line
-	1500 4750 1250 4750
-Connection ~ 1250 4750
-Wire Wire Line
-	1250 4750 1250 4550
 Wire Wire Line
 	1250 5500 900  5500
@@
 	3600 4400 3600 4850
 Connection ~ 3600 4850
+Wire Wire Line
+	1250 4550 1250 4900
 $EndSCHEMATC

Commit message: fixed resistor values for the 9V supply
Changed lines of the file:
@@
 F0 "Power" 50
 F1 "Power.sch" 50
-F2 "+12V" I L 8250 3400 50
-F3 "GND" I R 9300 3400 50
-F4 "+5V" I L 8250 3700 50
-F5 "+9V" I L 8250 3550 50
-F6 "-3.3V" I R 9300 3800 50
 $EndSheet
 $Comp

Commit message: ERC check on the schematics
Other:
- moved on the sheet: C1, J1, J2, J3, J4, J5, Q1, Q2, R1, R2, R3, R4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

Commit message: added footprints to components
Parts:
- TH1: footprint (none) -> Connector_PinHeader_2.54mm:PinHeader_1x02_P2.54mm_Vertical
- U1: value OPA2354 -> OPA2354AIDDA; footprint (none) -> Package_SO:SOIC-8-1EP_3.9x4.9mm_P1.27mm_EP2.29x3mm
Changed lines of the file:
@@
 F 0 "TH1" H 3855 5746 50  0000 L CNN
 F 1 "NTCALUG03A103G" H 3855 5655 50  0000 L CNN
-F 2 "" H 3750 5700 50  0001 C CNN
+F 2 "Connector_PinHeader_2.54mm:PinHeader_1x02_P2.54mm_Vertical" H 3750 5700 50  0001 C CNN
 F 3 "~" H 3750 5700 50  0001 C CNN
 	1    3750 5700
@@
 P 6350 5550
 F 0 "U1" H 6600 5687 60  0000 C CNN
-F 1 "OPA2354" H 6600 5581 60  0000 C CNN
-F 2 "" H 6400 5550 60  0001 C CNN
+F 1 "OPA2354AIDDA" H 6600 5581 60  0000 C CNN
+F 2 "Package_SO:SOIC-8-1EP_3.9x4.9mm_P1.27mm_EP2.29x3mm" H 6400 5550 60  0001 C CNN
 F 3 "" H 6400 5550 60  0001 C CNN
 	1    6350 5550
