File: Hardware/controller.sch (KiCad schematic (older format))
At the start: 6 parts, among them U2 Teensy4.0, U3 ADS7883SBDBVR

Commit message: removed labels from power connections. powr conn already global
Changed lines of the file:
@@
 Text HLabel 7150 4200 2    50   Input ~ 0
 TempSense
-Text HLabel 7850 3900 2    50   Input ~ 0
+Text HLabel 8100 3900 2    50   Input ~ 0
 ADC-SHUNT
 Wire Wire Line
@@
 L power:+3.3V #PWR0110
 U 1 1 5F784B57
-P 7150 2800
-F 0 "#PWR0110" H 7150 2650 50  0001 C CNN
-F 1 "+3.3V" H 7165 2973 50  0000 C CNN
-F 2 "" H 7150 2800 50  0001 C CNN
-F 3 "" H 7150 2800 50  0001 C CNN
-	1    7150 2800
+P 8050 2800
+F 0 "#PWR0110" H 8050 2650 50  0001 C CNN
+F 1 "+3.3V" H 8065 2973 50  0000 C CNN
+F 2 "" H 8050 2800 50  0001 C CNN
+F 3 "" H 8050 2800 50  0001 C CNN
+	1    8050 2800
 	1    0    0    -1
 $EndComp
-Wire Wire Line
-	6950 2800 7150 2800
-Text GLabel 7500 2800 1    50   Input ~ 0
-+3.3V
-Connection ~ 7150 2800
-Wire Wire Line
-	7150 2800 7650 2800
 $Comp
 L Analog_ADC:ADS7866 U3
@@
 NoConn ~ 6950 2400
 NoConn ~ 6950 2300
+Connection ~ 8050 2800
+Wire Wire Line
+	6950 2800 7650 2800
+Wire Wire Line
+	8100 3900 7850 3900
+Connection ~ 7850 3900
 $EndSCHEMATC

Commit message: fixed resistor values for the 9V supply
Connections:
- no-connect marks 23 -> 24
Changed lines of the file:
@@
 	8100 3900 7850 3900
 Connection ~ 7850 3900
+NoConn ~ 4750 3700
 $EndSCHEMATC

Commit message: ERC check on the schematics
Changed lines of the file:
@@
 $EndComp
-Wire Wire Line
-	6950 3000 7300 3000
 Wire Wire Line
 	6950 4700 7550 4700
@@
 L power:+3.3V #PWR0110
 U 1 1 5F784B57
-P 8050 2800
-F 0 "#PWR0110" H 8050 2650 50  0001 C CNN
-F 1 "+3.3V" H 8065 2973 50  0000 C CNN
-F 2 "" H 8050 2800 50  0001 C CNN
-F 3 "" H 8050 2800 50  0001 C CNN
-	1    8050 2800
+P 8050 2700
+F 0 "#PWR0110" H 8050 2550 50  0001 C CNN
+F 1 "+3.3V" H 8065 2873 50  0000 C CNN
+F 2 "" H 8050 2700 50  0001 C CNN
+F 3 "" H 8050 2700 50  0001 C CNN
+	1    8050 2700
 	1    0    0    -1
 $EndComp
@@
 U 1 1 5FCB3601
 P 3100 3700
-F 0 "U3" H 3100 4181 50  0000 C CNN
-F 1 "ADS7883SBDBVR" H 3100 4090 50  0000 C CNN
+F 0 "U3" H 3200 4100 50  0000 C CNN
+F 1 "ADS7883SBDBVR" H 3450 4000 50  0000 C CNN
 F 2 "Package_TO_SOT_SMD:TSOT-23-6" H 3100 3650 50  0001 C CNN
 F 3 "http://www.ti.com/lit/ds/symlink/ads7866.pdf" H 3150 3950 50  0001 C CNN
@@
 Connection ~ 7850 3900
 NoConn ~ 4750 3700
+Wire Wire Line
+	8050 2700 8050 2800
+Wire Wire Line
+	6950 3000 7300 3000
 $EndSCHEMATC

Commit message: added footprints to components
Parts:
- U2: footprint (none) -> Hardware:Teensy40
Changed lines of the file:
@@
 F 0 "U2" H 5850 5265 50  0000 C CNN
 F 1 "Teensy4.0" H 5850 5174 50  0000 C CNN
-F 2 "" H 5450 3850 50  0001 C CNN
+F 2 "Hardware:Teensy40" H 5450 3850 50  0001 C CNN
 F 3 "" H 5450 3850 50  0001 C CNN
 	1    5850 3650

Commit message: added footprints to missing parts. did rough placement
Parts:
- R35, R9: footprint (none) -> Resistor_SMD:R_0603_1608Metric
- U2: footprint Hardware:Teensy40 -> Hardware:Teensy40_SMT
Changed lines of the file:
@@
 F 0 "U2" H 5850 5265 50  0000 C CNN
 F 1 "Teensy4.0" H 5850 5174 50  0000 C CNN
-F 2 "Hardware:Teensy40" H 5450 3850 50  0001 C CNN
+F 2 "Hardware:Teensy40_SMT" H 5450 3850 50  0001 C CNN
 F 3 "" H 5450 3850 50  0001 C CNN
 	1    5850 3650
@@
 F 0 "R35" H 7920 4296 50  0000 L CNN
 F 1 "0R" H 7920 4205 50  0000 L CNN
-F 2 "" V 7780 4250 50  0001 C CNN
+F 2 "Resistor_SMD:R_0603_1608Metric" V 7780 4250 50  0001 C CNN
 F 3 "~" H 7850 4250 50  0001 C CNN
 	1    7850 4250
@@
 F 0 "R9" V 7193 3900 50  0000 C CNN
 F 1 "0R" V 7284 3900 50  0000 C CNN
-F 2 "" V 7330 3900 50  0001 C CNN
+F 2 "Resistor_SMD:R_0603_1608Metric" V 7330 3900 50  0001 C CNN
 F 3 "~" H 7400 3900 50  0001 C CNN
 	1    7400 3900
