File: Hardware/Laser-Driver-v3.kicad_pcb (KiCad board)
At the start: 2 copper layers, 67 parts, among them J1 Screw_Terminal_01x02, Q1 IRFP4568PbF, Q2 PSMN0R7-25YLD, Q3 BSS138, U10 LM2734Y, U11 LM285D-1.2, U16 TC4452, U3 ADS7883SBDBVR, U4 AD9744, U7 LM285M-ADJ, U8 LM2734Y

Commit message: added footprints to components
Parts:
- added C18: DNM, Capacitor_SMD:C_0603_1608Metric, F.Cu at (191.8, 110.7)
- added C2: 2.2uF, Capacitor_SMD:C_0603_1608Metric, F.Cu at (177.4, 118.2)
- added C3: 22uF, Capacitor_SMD:C_0805_2012Metric, F.Cu at (168.7, 118.5)
- added C4: 1000pF, Capacitor_SMD:C_0603_1608Metric, F.Cu at (181.4, 118.2)
- added C5: 22uF, Capacitor_SMD:C_0805_2012Metric, F.Cu at (173.2, 118.5)
- added D7: MBR0520, Diode_SMD:D_SOD-123, F.Cu at (155.4, 114.7)
- added J6: 694106301002, Connector_BarrelJack:BarrelJack_Wuerth_6941xx301002, F.Cu at (189.6, 90.0)
- added L3: 22uH, Inductor_SMD:L_Taiyo-Yuden_NR-60xx_HandSoldering, F.Cu at (171.3, 113.2)
- added L4: 22uH, Inductor_SMD:L_Taiyo-Yuden_NR-60xx_HandSoldering, F.Cu at (180.8, 113.2)
- added SW1: TL3305A, Button_Switch_SMD:SW_SPST_TL3305A, F.Cu at (109.6, 66.4)
- added TH1: NTCALUG03A103G, Connector_PinHeader_2.54mm:PinHeader_1x02_P2.54mm_Vertical, F.Cu at (138.7, 65.7)
- added U1: OPA2354AIDDA, Package_SO:SOIC-8-1EP_3.9x4.9mm_P1.27mm_EP2.29x3mm, F.Cu at (132.2, 66.6)
- added U12: 74LVC2G04, Package_TO_SOT_SMD:SOT-23-6_Handsoldering, F.Cu at (117.7, 65.7)
- added U13: SN74LVC1G08DBVR, Package_TO_SOT_SMD:SOT-23-5_HandSoldering, F.Cu at (113.9, 71.8)
- added U14: TC75S57FU(TE85L,F), Package_TO_SOT_SMD:SOT-353_SC-70-5, F.Cu at (122.8, 65.3)
- added U15: 74LVC2G02, Package_SO:SSOP-8_2.95x2.8mm_P0.65mm, F.Cu at (107.7, 71.6)
- added U2: Teensy4.0, Hardware:Teensy40, F.Cu at (175.4, 68.7)
- added U5: THS3091, Package_SO:SOIC-8_3.9x4.9mm_P1.27mm, F.Cu at (167.4, 89.1)
- added U6: THS3091, Package_SO:SOIC-8_3.9x4.9mm_P1.27mm, F.Cu at (175.8, 89.1)
- added U9: LM2611xMF, Package_TO_SOT_SMD:SOT-23-5, F.Cu at (160.7, 115.3)
- C25: value 10uF -> 10uF 25V
- C26: value 10nF -> 10nF 16V
- C27: value 22uF -> 22uF 16V
- L1: value SRR0604-100ML -> 4.7uH 1.2A
- L2: value SLF7032T-6R8M1R -> 22uH 1.4 A
- R16: value 25R -> 16.83k 1%
- R17: value 25R -> 10k 1%
- R24, R27: value 10k -> 10k 1%
- R25: value 10k -> 100k
- R26: value 10k -> 102k 1%
- moved J1 115.4 mm to (123.7, 123.1)
- moved U3 108.8 mm to (171.1, 103.1)
- moved C16 108.8 mm to (175.8, 104.6)
- moved R17 106.9 mm to (158.5, 118.9)
- moved C17 100.8 mm to (142.1, 112.1)
- moved C19 100.8 mm to (146.8, 109.6)
- moved C20 100.8 mm to (151.3, 100.6)
- moved R11 100.8 mm to (151.3, 103.1)
- moved R12 100.8 mm to (146.8, 107.1)
- moved R14 100.8 mm to (138.1, 112.1)
- moved R15 100.8 mm to (130.1, 111.9)
- moved R19 100.8 mm to (134.1, 111.9)
- moved R28 100.8 mm to (153.2, 89.7)
- moved R32 100.8 mm to (153.2, 84.6)
- moved R33 100.8 mm to (136.7, 94.0)
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Connections:
- C19 pad 2: Net-(C19-Pad2) -> +9V
- C30 pad 1: GND -> +5V
- C30 pad 2: +5V -> GND
- Q3 pad 3: Net-(Q3-Pad3) -> /Overcurrent Protection/OCStatus
- R15 pad 2: /Output Stage/MOSFET-OUT -> Net-(R15-Pad2)
- R16 pad 1: /Output Stage/MOSFET-OUT -> -3V3
- R16 pad 2: +9V -> Net-(C4-Pad1)
- R17 pad 1: /Output Stage/MOSFET-OUT -> Net-(C4-Pad1)
- R17 pad 2: Net-(C19-Pad2) -> GND
- R18 pad 1: Net-(R18-Pad1) -> Net-(R14-Pad2)
- R18 pad 2: Net-(R14-Pad2) -> Net-(R18-Pad2)
- R19 pad 1: Net-(R18-Pad1) -> Net-(R18-Pad2)
- R2 pad 1: (no net) -> /Overcurrent Protection/OCSense
- R21 pad 2: Net-(R18-Pad1) -> Net-(R18-Pad2)
- R3 pad 1: (no net) -> /Teensy/ADC-SHUNT
- R30 pad 2: (no net) -> Net-(R30-Pad2)
- R32 pad 1: Net-(Q3-Pad3) -> Net-(R32-Pad1)
- R33 pad 1: (no net) -> /Overcurrent Protection/OCStatus
- R33 pad 2: Net-(Q3-Pad3) -> Net-(R32-Pad1)
- R4 pad 2: (no net) -> Net-(R4-Pad2)
- U16 pad 2: Net-(Q3-Pad3) -> Net-(R32-Pad1)
- U3 pad 4: (no net) -> Net-(U2-Pad20)
- U3 pad 5: (no net) -> Net-(U2-Pad14)
- U3 pad 6: (no net) -> Net-(U2-Pad12)
- U4 pad 1: (no net) -> /Output Stage/DAC-D13
- U4 pad 10: (no net) -> /Output Stage/DAC-D4
- U4 pad 11: (no net) -> /Output Stage/DAC-D3
- U4 pad 12: (no net) -> /Output Stage/DAC-D2
- U4 pad 13: (no net) -> /Output Stage/DAC-D1
- U4 pad 14: (no net) -> /Output Stage/DAC-D0
- U4 pad 2: (no net) -> /Output Stage/DAC-D12
- U4 pad 28: (no net) -> /Output Stage/DAC-CLOCK
- U4 pad 3: (no net) -> /Output Stage/DAC-D11
- U4 pad 4: (no net) -> /Output Stage/DAC-D10
- U4 pad 5: (no net) -> /Output Stage/DAC-D9
- U4 pad 6: (no net) -> /Output Stage/DAC-D8
- U4 pad 7: (no net) -> /Output Stage/DAC-D7
- U4 pad 8: (no net) -> /Output Stage/DAC-D6
- U4 pad 9: (no net) -> /Output Stage/DAC-D5
- U7 pad 8: Net-(R18-Pad1) -> Net-(R18-Pad2)

Commit message: added footprints to missing parts. did rough placement
Parts:
- removed TH1: NTCALUG03A103G, Connector_PinHeader_2.54mm:PinHeader_1x02_P2.54mm_Vertical
- added J2: 74650074R, Hardware:7460307, F.Cu at (168.0, 50.0)
- added J5: 74650074R, Hardware:7460307, F.Cu at (99.9, 50.7)
- added R35: 0R, Resistor_SMD:R_0603_1608Metric, F.Cu at (179.5, 76.6)
- added R7: 1 mOhms ±5% 10W, Hardware:2959_metric_15075, F.Cu at (118.0, 51.0)
- added R9: 0R, Resistor_SMD:R_0603_1608Metric, F.Cu at (51.2, 123.7)
- U2: footprint Hardware:Teensy40 -> Hardware:Teensy40_SMT
- moved Q3 95.5 mm to (80.8, 143.2)
- moved R32 95.5 mm to (80.6, 146.7)
- moved C16 86.8 mm to (260.6, 86.2)
- moved R15 86.8 mm to (214.9, 93.5)
- moved R19 86.8 mm to (218.9, 93.5)
- moved R20 86.8 mm to (232.1, 82.2)
- moved R21 86.8 mm to (223.6, 88.7)
- moved C1 86.8 mm to (193.0, 88.8)
- moved R13 86.8 mm to (227.6, 91.2)
- moved R18 86.8 mm to (223.6, 91.2)
- moved R2 86.8 mm to (193.0, 96.3)
- moved R3 86.8 mm to (193.0, 93.8)
- moved R4 86.8 mm to (197.0, 91.3)
- moved R5 86.8 mm to (207.3, 82.2)
- moved R8 86.8 mm to (198.9, 88.8)
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Connections:
- Q1 pad 2: (no net) -> Net-(J2-Pad1)
- R4 pad 1: (no net) -> Net-(Q2-Pad1)
- R5 pad 2: (no net) -> GND
- U2 pad 38: (no net) -> Net-(R9-Pad2)
- U3 pad 3: (no net) -> Net-(R35-Pad2)
Other:
- board outline added: 90 x 80 mm

Commit message: finished placement. started routing
Parts:
- added C6: 100nF, Capacitor_SMD:C_0603_1608Metric, F.Cu at (110.2, 90.0)
- added C7: 100nF, Capacitor_SMD:C_0603_1608Metric, F.Cu at (161.4, 84.0)
- added C8: 100nF, Capacitor_SMD:C_0603_1608Metric, F.Cu at (165.2, 79.8)
- added D8: RED, LED_SMD:LED_0603_1608Metric, F.Cu at (132.1, 117.3)
- added H1: M3, MountingHole:MountingHole_3.2mm_M3_Pad_Via, F.Cu at (175.0, 115.0)
- added H2: M3, MountingHole:MountingHole_3.2mm_M3_Pad_Via, F.Cu at (95.0, 115.0)
- added H3: M3, MountingHole:MountingHole_3.2mm_M3_Pad_Via, F.Cu at (175.0, 45.0)
- added H4: M3, MountingHole:MountingHole_3.2mm_M3_Pad_Via, F.Cu at (95.0, 45.0)
- added HS1: Heatsink, Heatsink:Heatsink_Aavid-TV5G_TO220_Horizontal, F.Cu at (143.0, 57.0)
- added R36: 1k, Resistor_SMD:R_0603_1608Metric, F.Cu at (132.1, 114.0)
- C21, C27: footprint Capacitor_SMD:C_0603_1608Metric -> Capacitor_SMD:C_0805_2012Metric
- C23: footprint Capacitor_SMD:C_0603_1608Metric -> Capacitor_SMD:C_1206_3216Metric
- C3, C5: footprint Capacitor_SMD:C_0805_2012Metric -> Capacitor_SMD:C_1206_3216Metric
- D2, D4: value SS1P3L -> CRS08; footprint Diode_SMD:D_SMA -> Diode_SMD:D_SOD-123F
- D6: value TLLR4400 -> GREEN; footprint LED_THT:LED_D3.0mm -> LED_SMD:LED_0603_1608Metric
- L1: footprint Inductor_SMD:L_6.3x6.3_H3 -> Inductor_SMD:L_Taiyo-Yuden_NR-40xx
- L2: value 22uH 1.4 A -> 22uH 1.4A; footprint Inductor_SMD:L_7.3x7.3_H3.5 -> Inductor_SMD:L_Taiyo-Yuden_NR-50xx
- L3, L4: value 22uH -> 22uH 1.4A; footprint Inductor_SMD:L_Taiyo-Yuden_NR-60xx_HandSoldering -> Inductor_SMD:L_Taiyo-Yuden_NR-50xx
- R31: value 1,55K -> 1k
- RV1: footprint Potentiometer_THT:Potentiometer_ACP_CA9-V10_Vertical -> Potentiometer_SMD:Potentiometer_Bourns_3314G_Vertical
- moved C19 98.2 mm to (134.0, 80.8), turned to 90 degrees
- moved C16 96.0 mm to (168.6, 113.6)
- moved R5 93.6 mm to (113.8, 78.4), turned to 90 degrees
- moved C20 92.3 mm to (143.8, 81.0), turned to 90 degrees
- moved R9 89.2 mm to (134.8, 92.6)
- moved R8 86.7 mm to (112.8, 99.2), turned to 180 degrees
- moved R4 82.6 mm to (115.4, 78.4), turned to 270 degrees
- moved R32 82.6 mm to (139.2, 88.5), turned to 270 degrees
- moved R3 80.3 mm to (112.8, 97.6)
- moved R6 79.2 mm to (113.9, 87.5)
- moved R33 78.5 mm to (137.6, 88.5), turned to 90 degrees
- moved R2 77.7 mm to (115.3, 98.4), turned to 90 degrees
- moved Q3 76.7 mm to (134.7, 88.7)
- moved R11 76.4 mm to (160.2, 75.7), turned to 270 degrees
- moved R20 75.6 mm to (157.1, 72.5), turned to 270 degrees
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Connections:
- R6 pad 1: Net-(R5-Pad1) -> Net-(R2-Pad2)
- R6 pad 2: Net-(R2-Pad2) -> Net-(R5-Pad1)
- U1 pad 1: Net-(R2-Pad2) -> /Teensy/ADC-SHUNT
- U1 pad 2: Net-(R5-Pad1) -> Net-(R3-Pad2)
- U1 pad 3: Net-(R4-Pad2) -> Net-(R2-Pad2)
- U1 pad 5: Net-(R2-Pad2) -> Net-(R4-Pad2)
- U1 pad 6: Net-(R3-Pad2) -> Net-(R5-Pad1)
- U1 pad 7: /Teensy/ADC-SHUNT -> Net-(R2-Pad2)
Routing:
- net +9V: track 0.00 -> 32.8 mm, vias 0 -> 3
- net +12V: track 0.00 -> 27.8 mm, vias 0 -> 5
- net GND: track 0.00 -> 22.9 mm, vias 0 -> 16
- net +5V: track 0.00 -> 22.4 mm, vias 0 -> 3
- net Net-(C26-Pad2): track 0.00 -> 15.3 mm
- net -3V3: track 0.00 -> 10.4 mm, vias 0 -> 2
- net Net-(C2-Pad1): track 0.00 -> 8.05 mm
- net Net-(C4-Pad1): track 0.00 -> 6.77 mm
- net Net-(C22-Pad2): track 0.00 -> 6.38 mm
- net Net-(C22-Pad1): track 0.00 -> 5.55 mm
- net Net-(C2-Pad2): track 0.00 -> 5.43 mm
- net Net-(C26-Pad1): track 0.00 -> 5.12 mm
- net Net-(R23-Pad2): track 0.00 -> 4.20 mm
- net Net-(R26-Pad2): track 0.00 -> 3.74 mm
- net Net-(R25-Pad2): track 0.00 -> 3.35 mm
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- added copper zone on In1.Cu, net GND
Other:
- outline, holes or cut-outs redrawn
- copper layers 2 -> 4

Commit message: finished pcb
Parts:
- added C9: 100nF, Capacitor_SMD:C_0603_1608Metric, F.Cu at (175.0, 75.3)
- added R37: 1M, Resistor_SMD:R_0603_1608Metric, F.Cu at (175.1, 77.0)
- HS1: footprint Heatsink:Heatsink_Aavid-TV5G_TO220_Horizontal -> Hardware:RA-T2X-38E
- moved Q1 9.05 mm to (148.7, 53.5), turned to 180 degrees
- moved R4 7.72 mm to (109.3, 73.6)
- moved R5 7.72 mm to (107.8, 73.6)
- moved Q2 7.60 mm to (117.8, 58.7)
- moved R7 5.50 mm to (108.5, 58.2)
- moved C5 4.79 mm to (104.4, 99.3)
- moved D7 4.79 mm to (94.4, 100.8)
- moved J6 4.79 mm to (105.9, 82.8)
- moved R16 4.79 mm to (104.2, 95.8)
- moved R17 4.79 mm to (104.2, 92.6)
- moved U9 4.79 mm to (100.2, 95.2)
- moved C3 4.79 mm to (100.6, 91.6)
- moved C4 4.79 mm to (105.8, 95.8)
- moved C2 4.79 mm to (94.0, 97.4)
- moved L3 4.79 mm to (95.2, 93.4)
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Connections:
- H1 pad 1: GND -> Earth
- H2 pad 1: GND -> Earth
- H3 pad 1: GND -> Earth
- H4 pad 1: GND -> Earth
Routing:
- net GND: track 22.9 -> 132.4 mm, vias 16 -> 82
- net +5V: track 22.4 -> 103.2 mm, vias 3 -> 18
- net +3V3: track 0.00 -> 75.7 mm, vias 0 -> 8
- net +12V: track 27.8 -> 90.6 mm, vias 5 -> 6
- net /Output Stage/DAC-D10: track 0.00 -> 45.7 mm, vias 0 -> 1
- net /Teensy/ADC-SHUNT: track 0.00 -> 42.6 mm
- net /Output Stage/MOSFET-OUT: track 0.00 -> 40.6 mm, vias 0 -> 1
- net /Output Stage/DAC-D11: track 0.00 -> 40.0 mm, vias 0 -> 1
- net /Overcurrent Protection/OCControl: track 0.00 -> 38.0 mm, vias 0 -> 2
- net Net-(R31-Pad2): track 0.00 -> 38.0 mm, vias 0 -> 2
- net /Output Stage/DAC-CLOCK: track 0.00 -> 35.4 mm, vias 0 -> 1
- net /Output Stage/DAC-D12: track 0.00 -> 33.7 mm, vias 0 -> 1
- net Earth: track 0.00 -> 32.4 mm
- net /Teensy/TempSense: track 0.00 -> 26.6 mm
- net /Output Stage/DAC-D13: track 0.00 -> 26.6 mm, vias 0 -> 1
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- added copper zone on In2.Cu, net +12V
- added copper zone on In2.Cu, net +3V3
- added copper zone on B.Cu, net +5V
- added copper zone on In2.Cu, net +5V
- added copper zone on In2.Cu, net +9V
- added copper zone on B.Cu, net Earth
- added copper zone on F.Cu, net Earth
- added copper zone on In1.Cu, net Earth
- added copper zone on In2.Cu, net Earth
- added copper zone on B.Cu, net GND
- added copper zone on F.Cu, net GND
- added copper zone on In2.Cu, net GND
- added copper zone on B.Cu, net Net-(J2-Pad1)
- added copper zone on F.Cu, net Net-(J2-Pad1)
- added copper zone on In1.Cu, net Net-(J2-Pad1)
- added copper zone on In2.Cu, net Net-(J2-Pad1)
- added copper zone on B.Cu, net Net-(Q1-Pad3)
- added copper zone on F.Cu, net Net-(Q1-Pad3)
- added copper zone on In1.Cu, net Net-(Q1-Pad3)
- added copper zone on In2.Cu, net Net-(Q1-Pad3)
- added copper zone on B.Cu, net Net-(Q2-Pad1)
- added copper zone on F.Cu, net Net-(Q2-Pad1)
- added copper zone on In1.Cu, net Net-(Q2-Pad1)
- added copper zone on In2.Cu, net Net-(Q2-Pad1)

Commit message: changed heatsink
Parts:
- HS1: value Heatsink -> ATS-1139-C1-R0; footprint Hardware:RA-T2X-38E -> Hardware:ATS-1141; moved to B.Cu
- J2, J5: value 74650074R -> 7460307
- Q1: moved to B.Cu
- moved U7 23.5 mm to (141.8, 75.4), turned to 0 degrees
- moved Q1 11.5 mm to (140.4, 45.5)
- moved R15 10.4 mm to (141.6, 85.4)
- moved HS1 9.02 mm to (135.0, 60.0)
- moved R5 7.55 mm to (111.5, 80.2), turned to 180 degrees
- moved R11 6.89 mm to (152.3, 78.4)
- moved R12 6.89 mm to (150.0, 83.9)
- moved R13 6.89 mm to (150.0, 82.2)
- moved R14 6.89 mm to (150.0, 80.7)
- moved R18 6.89 mm to (150.0, 79.1)
- moved R19 6.89 mm to (150.8, 75.2)
- moved R20 6.89 mm to (149.2, 75.2)
- moved R21 6.89 mm to (150.0, 77.5)
- moved C18 6.89 mm to (152.3, 81.5)
- moved C20 6.70 mm to (137.0, 84.5)
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Routing:
- net Earth: track 32.4 -> 14.7 mm
- net GND: track 132.4 -> 148.3 mm, vias 82 -> 76
- net Net-(Q2-Pad1): track 15.8 -> 30.9 mm, vias 28 -> 16
- net +12V: track 90.6 -> 79.2 mm
- net Net-(C18-Pad2): track 15.0 -> 22.7 mm
- net Net-(C18-Pad1): track 15.4 -> 23.0 mm
- net Net-(R13-Pad2): track 15.8 -> 9.64 mm
- net Net-(R5-Pad1): track 18.5 -> 13.2 mm
- net Net-(R4-Pad2): track 18.6 -> 13.8 mm
- net Net-(R18-Pad2): track 10.3 -> 14.6 mm
- net Net-(R14-Pad2): track 8.63 -> 6.66 mm
- net Net-(R19-Pad2): track 10.0 -> 8.43 mm
- net +9V: track 40.6 -> 39.3 mm
- net Net-(R15-Pad2): track 15.0 -> 15.8 mm
