File: Hardware/Laser-Driver-v3.kicad_pcb (KiCad board)
At the start: 4 copper layers, 90 x 80 mm, 103 parts, among them J1 Screw_Terminal_01x02, J2 7460307, J5 7460307, J6 694106301002, Q1 IRFP4568PbF, Q2 PSMN0R7-25YLD, Q3 BSS138, SW1 TL3305A, U1 OPA2354AIDDA, U10 LM2734Y, U11 LM285D-1.2, U12 74LVC2G04, U13 SN74LVC1G08DBVR, U14 TC75S57FU(TE85L,F), U15 74LVC2G02, U16 TC4452, U2 Teensy4.0, U3 ADS7883SBDBVR, U4 AD9744, U5 THS3091, U6 THS3091, U7 LM285M-ADJ, U8 LM2734Y, U9 LM2611xMF

Commit message: moved MOSFET to the middle, removed heatsink
Parts:
- removed HS1: ATS-1139-C1-R0, Hardware:ATS-1141
- moved Q1 17.1 mm to (140.5, 62.6)
Routing:
- net /Output Stage/MOSFET-OUT: track 41.0 -> 24.0 mm
